File: hardware/MC34063A.kicad_sch (KiCad schematic)
At the start: 17 parts, among them Q201 MPSA92, Q202 P4NK60ZFP, U201 MC34063AP

Commit message: MAX1771
Parts:
- added J201: INPUT, TerminalBlock_Phoenix:TerminalBlock_Phoenix_MKDS-1,5-2-5.08_1x02_P5.08mm_Horizontal, symbol Connector:Screw_Terminal_01x02
- added J202: OUTPUT, TerminalBlock_Phoenix:TerminalBlock_Phoenix_MKDS-1,5-2-5.08_1x02_P5.08mm_Horizontal, symbol Connector:Screw_Terminal_01x02
- added NT201: GND_PWR_GND, NetTie:NetTie-2_SMD_Pad0.5mm, symbol Device:NetTie_2
- added NT202: IN_PWN_IN, NetTie:NetTie-2_SMD_Pad0.5mm, symbol Device:NetTie_2
- added NT203: 12V_SENSE, NetTie:NetTie-2_SMD_Pad0.5mm, symbol Device:NetTie_2
- added NT204: OUT_FEEDBACK, NetTie:NetTie-2_SMD_Pad0.5mm, symbol Device:NetTie_2
- C201, C203: footprint Capacitor_THT:C_Disc_D5.0mm_W2.5mm_P2.50mm -> Capacitor_THT:C_Disc_D5.0mm_W2.5mm_P5.00mm
- C202: footprint Capacitor_THT:CP_Radial_D8.0mm_P3.80mm -> Capacitor_THT:CP_Radial_D8.0mm_P5.00mm
- C204: renamed from C205; footprint Capacitor_THT:C_Disc_D5.0mm_W2.5mm_P2.50mm -> Capacitor_THT:C_Disc_D5.0mm_W2.5mm_P5.00mm
- D201, D202: footprint Diode_THT:D_DO-41_SOD81_P10.16mm_Horizontal -> Diode_THT:D_DO-41_SOD81_P7.62mm_Horizontal
- Q201: footprint Package_TO_SOT_THT:TO-92_Inline -> Package_TO_SOT_THT:TO-92_Inline_Wide
- R201, R202, R203, R204, R205: footprint Resistor_THT:R_Axial_DIN0207_L6.3mm_D2.5mm_P10.16mm_Horizontal -> Resistor_THT:R_Axial_DIN0207_L6.3mm_D2.5mm_P7.62mm_Horizontal
- renumbered C204 to C205
Connections:
- net +12V: now also J201.2 (Pin_2), NT202.1; no longer U201.6 (Vin)
- net +170V: now also J202.1 (Pin_1), NT204.2; no longer VR201.2
- net GND: now also NT201.2; no longer C201.2, C202.2, C205.2, Q201.1 (E), Q202.3 (S), R203.1
- net at D201.1 (K), Q202.1 (G): now also Q201.1 (E); no longer Q201.3 (C)
- net INDUCTOR_OUT: now reaches D202.2 (A), L201.2, Q202.2 (D)
- net at U201.1 (SwC), U201.7 (Ipk), U201.8 (DC): now also NT203.1; no longer L201.1, R201.2
- new net: NT204.1, VR201.2
- new net: NT202.2, U201.6 (Vin)
- new net INDUCTOR_IN: L201.1, NT203.2, R201.2
- new net PWR_GND: C201.2, C202.2, C205.2, J201.1 (Pin_1), J202.2 (Pin_2), NT201.1, Q201.3 (C), Q202.3 (S), R203.1
Other:
- moved on the sheet: C201, C202, C205
