File: hardware/NosClock.kicad_sch (KiCad schematic)
At the start: 0 parts

Commit message: MC34063
Other:
- added sheet MC34063A (MC34063A.kicad_sch)
Changed lines of the file:
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@@
 	(generator_version "9.0")
 	(paper "A4")
+	(sheet
+		(at 195.58 118.11)
+		(size 29.21 17.78)
+		(exclude_from_sim no)
+		(in_bom yes)
+		(on_board yes)
+		(dnp no)
+		(fields_autoplaced yes)
+		(stroke
+			(width 0.1524)
+			(type solid)
+		)
+		(fill
+			(color 0 0 0 0.0000)
+		)
+		(property "Sheetname" "MC34063A"
+			(at 195.58 117.3984 0)
+			(effects
+				(font
+					(size 1.27 1.27)
+				)
+				(justify left bottom)
+			)
+		)
+		(property "Sheetfile" "MC34063A.kicad_sch"
+			(at 195.58 136.4746 0)
+			(effects
+				(font
+					(size 1.27 1.27)
+				)
+				(justify left top)
+			)
+		)
+		(instances
+			(project "NosClock"
+				(path "/5a46aee9-b968-477e-a4a1-4edba06163a3"
+					(page "2")
+				)
+			)
+		)
+	)
 	(sheet_instances
 		(path "/"

Commit message: MAX1771
Parts:
- added C103: 100uF 10V, Capacitor_THT:CP_Radial_D6.3mm_P2.50mm, symbol Device:C_Polarized
- added NX101: ~, nixies-us:nixies-us-IN-12-DSUB, symbol nixies-us:IN-12BORIGINAL
- added R101: 10K, Resistor_SMD:R_2512_6332Metric_Pad1.40x3.35mm_HandSolder, symbol Device:R
- added TP101: A, TestPoint:TestPoint_Pad_3.0x3.0mm, symbol Connector:TestPoint
- added TP102: B, TestPoint:TestPoint_Pad_3.0x3.0mm, symbol Connector:TestPoint
- added TP103: C, TestPoint:TestPoint_Pad_3.0x3.0mm, symbol Connector:TestPoint
- added TP104: D, TestPoint:TestPoint_Pad_3.0x3.0mm, symbol Connector:TestPoint
- added TP105: 5V, TestPoint:TestPoint_Pad_3.0x3.0mm, symbol Connector:TestPoint
- added U101: К155ИД1, Package_DIP:DIP-16_W7.62mm, symbol 74xx_IEEE:74141
- added U102: AMS1117-5, Package_TO_SOT_SMD:SOT-223-3_TabPin2, symbol Regulator_Linear:AMS1117-3.3
Connections:
- new net: TP102.1, U101.6 (B)
- new net: TP103.1, U101.7 (C)
- new net: NX101.0, U101.16 (~{Q0})
- new net: NX101.1, U101.15 (~{Q1})
- new net: NX101.2, U101.8 (~{Q2})
- new net: NX101.3, U101.9 (~{Q3})
- new net: NX101.4, U101.13 (~{Q4})
- new net: NX101.5, U101.14 (~{Q5})
- new net: NX101.6, U101.11 (~{Q6})
- new net: NX101.7, U101.10 (~{Q7})
- new net: NX101.8, U101.1 (~{Q8})
- new net: NX101.9, U101.2 (~{Q9})
- new net: NX101.A, R101.1
- new net: TP101.1, U101.3 (A)
- new net: TP104.1, U101.4 (D)
- new net 12V: U102.3 (VI)
- new net 5V: C103.1, TP105.1, U101.5 (VCC), U102.2 (VO)
- new net GND: C103.2, U102.1 (GND)
- new net MAX1771/170V: R101.2
- new net MAX1771/PWR_GND: U101.12 (GND)
- no-connect marks 0 -> 1
Other:
- added sheet MAX1771 (MAX1771.kicad_sch)
- note added: "LDO"

Commit message: UC3843
Parts:
- added TP104: GND, TestPoint:TestPoint_Pad_3.0x3.0mm, symbol Connector:TestPoint
- added TP107: 12V, TestPoint:TestPoint_Pad_3.0x3.0mm, symbol Connector:TestPoint
- added TP108: 170V, TestPoint:TestPoint_Pad_3.0x3.0mm, symbol Connector:TestPoint
- renumbered C103 to C101, TP104 to TP101, TP105 to TP102, TP102 to TP105, TP101 to TP106, U102 to U101, U101 to U102
Connections:
- net 12V: now also TP107.1
- net MAX1771/170V renamed UC3843/170V
- net UC3843/170V: now also TP108.1
- net MAX1771/PWR_GND renamed UC3843/PWR_GND
- net UC3843/PWR_GND: now also TP104.1
Other:
- removed sheet MAX1771
- removed sheet MC34063A
- added sheet UC3843 (UC3843.kicad_sch)

Commit message: Lamps & 3.3v/5v
Parts:
- removed C101: 100uF 10V, Capacitor_THT:CP_Radial_D6.3mm_P2.50mm, symbol Device:C_Polarized
- removed NX101: ~, nixies-us:nixies-us-IN-12-DSUB, symbol nixies-us:IN-12BORIGINAL
- removed TP101: D, TestPoint:TestPoint_Pad_3.0x3.0mm, symbol Connector:TestPoint
- removed TP102: 5V, TestPoint:TestPoint_Pad_3.0x3.0mm, symbol Connector:TestPoint
- removed TP103: C, TestPoint:TestPoint_Pad_3.0x3.0mm, symbol Connector:TestPoint
- removed TP104: GND, TestPoint:TestPoint_Pad_3.0x3.0mm, symbol Connector:TestPoint
- removed TP105: B, TestPoint:TestPoint_Pad_3.0x3.0mm, symbol Connector:TestPoint
- removed TP106: A, TestPoint:TestPoint_Pad_3.0x3.0mm, symbol Connector:TestPoint
- removed TP107: 12V, TestPoint:TestPoint_Pad_3.0x3.0mm, symbol Connector:TestPoint
- removed TP108: 170V, TestPoint:TestPoint_Pad_3.0x3.0mm, symbol Connector:TestPoint
- removed U101: AMS1117-5, Package_TO_SOT_SMD:SOT-223-3_TabPin2, symbol Regulator_Linear:AMS1117-3.3
- removed U102: К155ИД1, Package_DIP:DIP-16_W7.62mm, symbol 74xx_IEEE:74141
- added C101: 1uF, Capacitor_SMD:C_0805_2012Metric, symbol Device:C
- added D101: ES1J, Diode_SMD:D_SMA_Handsoldering, symbol Device:D
- added J101: USB_C_Receptacle_USB2.0_16P, Connector_USB:USB_C_Receptacle_HRO_TYPE-C-31-M-12, symbol Connector:USB_C_Receptacle_USB2.0_16P
- added J102: AC, NosLib:TerminalBlock_Phoenix_MKDS-1,5-2-5.08_1x02_P5.08mm_Horizontal, symbol Connector:Screw_Terminal_01x02
- added NT101: NetTie_2, NetTie:NetTie-2_SMD_Pad0.5mm, symbol Device:NetTie_2
- added R102: 10K, Resistor_SMD:R_0603_1608Metric, symbol Device:R
- added R103, R104: 5.1K, Resistor_SMD:R_0603_1608Metric, symbol Device:R
- added R107: 4.7K, Resistor_SMD:R_0603_1608Metric, symbol Device:R
- added TP_101: BOOT, NosLib:TestPoint_Pad_1.0x1.0mm, symbol Connector:TestPoint
- added TP_102: EN, NosLib:TestPoint_Pad_1.0x1.0mm, symbol Connector:TestPoint
- added TP_103: GND, NosLib:TestPoint_Pad_1.0x1.0mm, symbol Connector:TestPoint
- added U102: ESP32-C3-WROOM-02, PCM_Espressif:ESP32-C3-WROOM-02, symbol PCM_Espressif:ESP32-C3-WROOM-02
- added U103: DS18B20, Package_TO_SOT_THT:TO-92_Inline, symbol Sensor_Temperature:DS18B20
- R101: footprint Resistor_SMD:R_2512_6332Metric_Pad1.40x3.35mm_HandSolder -> Resistor_SMD:R_0603_1608Metric
Connections:
- net 5V: now also NT101.2
- net GND: now also R101.2, C101.2, J101.A1 (GND), J101.A12 (GND), J101.B1 (GND), J101.B12 (GND), J101.S1 (SHIELD), J102.1 (Pin_1), R103.2, R104.2, TP_103.1, U102.19 (GND), U102.9 (GND), U103.1 (GND)
- net UC3843/170V: no longer R101.2
- net BOOT: now reaches R101.1
- net BOOT: now also TP_101.1, U102.8 (GPIO9)
- new net: J101.A4 (VBUS), J101.A9 (VBUS), J101.B4 (VBUS), J101.B9 (VBUS), NT101.1
- new net: J101.A5 (CC1), R103.1
- new net: J101.B5 (CC2), R104.1
- new net +12V: J102.2 (Pin_2)
- new net +3V3: R107.1, U102.1 (3V3), U103.3 (V_{DD})
- new net 3V3: R102.1
- new net CS: U102.10 (GPIO10)
- new net DALLAS: R107.2, U102.7 (GPIO8), U103.2 (DQ)
- new net EN: C101.1, R102.2, TP_102.1, U102.2 (EN/CHIP_PU)
- new net LED: U102.3 (GPIO4/ADC1_CH4)
- new net MOSI: U102.6 (GPIO7)
- new net SCK: U102.5 (GPIO6)
- new net TwoDigits1/FIRST_SK6812MINI_VCC: D101.1 (K)
- new net USB_D+: J101.A6 (D+), J101.B6 (D+), U102.14 (GPIO19/USB_D+)
- new net USB_D-: J101.A7 (D-), J101.B7 (D-), U102.13 (GPIO18/USB_D-)
- new net ~{PWM_DIGITS}: U102.15 (GPIO3/ADC1_CH3)
- new net ~{PWM_DOTS}: U102.4 (GPIO5/ADC2_CH0)
- no-connect marks 1 -> 7
Other:
- added sheet Dots (Dots.kicad_sch)
- added sheet LDO (LDO.kicad_sch)
- added sheet MP2307 (MP2307.kicad_sch)
- added sheet TwoDigits1 (TwoDigits.kicad_sch)
- added sheet TwoDigits2 (TwoDigits.kicad_sch)
- added sheet TwoDigits3 (TwoDigits.kicad_sch)
- note added: "DALLAS"
- note added: "ESP32 EN, BOOT"
- note added: "POWER"
- note added: "USB"
- note removed: "LDO"
