File: hardware/NosClock.kicad_sch (KiCad schematic)
At the start: 32 parts, among them J101 USB_C_Receptacle_USB2.0_16P, J102 Conn_01x02, J103 Conn_01x04, J104 12V IN, U101 ESP32-C3-MINI-1, U103 DS3231MZ

Commit message: hotfixes
Parts:
- TP_105: value SDA -> SCL/BOOT
- TP_107: value SCL/BOOT -> SDA
Changed lines of the file:
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@@
 			)
 		)
-		(property "Value" "SDA"
-			(at 240.538 148.59 90)
+		(property "Value" "SCL/BOOT"
+			(at 237.998 148.844 90)
 			(show_name no)
 			(do_not_autoplace no)
@@
 			)
 		)
-		(property "Value" "SCL/BOOT"
+		(property "Value" "SDA"
 			(at 240.538 153.67 90)
 			(show_name no)
