File: hardware/Dots.kicad_sch (KiCad schematic)
At the start: 2 parts, among them U101 74HC595

Commit message: Static version (incomplete)
Parts:
- removed R804: 10K, Resistor_SMD:R_0603_1608Metric, symbol Device:R
- added R901: 10K, Resistor_SMD:R_0603_1608Metric, symbol Device:R
- renumbered U101 to U901
Connections:
- net +3V3: now also R901.1
- net Dot1/EN: now also U901.2 (QC); no longer U901.1 (QB)
- net Dot2/EN: now also U901.3 (QD); no longer U901.2 (QC)
- net Dot3/EN: now also U901.1 (QB); no longer U901.3 (QD)
- net ~{PWM}: now also R901.2
