File: hardware/LDO.kicad_sch (KiCad schematic)
At the start: 5 parts, among them U301 AP7361-33ER-13

Commit message: Static version (incomplete)
Parts:
- removed C302: 10uF, Capacitor_SMD:C_0805_2012Metric, symbol Device:C
- renumbered C303 to C302, C304 to C303
Other:
- moved on the sheet: C301
Changed lines of the file:
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@@
-	)
-	(junction
-		(at 91.44 85.09)
-		(diameter 0)
-		(color 0 0 0 0)
 	)
 	(junction
@@
 	)
 	(junction
-		(at 91.44 97.79)
-		(diameter 0)
-		(color 0 0 0 0)
-	)
-	(junction
-		(at 76.2 85.09)
+		(at 87.63 85.09)
 		(diameter 0)
 		(color 0 0 0 0)
@@
 	(wire
 		(pts
-			(xy 91.44 85.09) (xy 97.79 85.09)
-		)
-		(stroke
-			(width 0)
-			(type default)
-		)
-	)
-	(wire
-		(pts
-			(xy 67.31 85.09) (xy 76.2 85.09)
+			(xy 87.63 85.09) (xy 97.79 85.09)
+		)
+		(stroke
+			(width 0)
+			(type default)
+		)
+	)
+	(wire
+		(pts
+			(xy 78.74 85.09) (xy 87.63 85.09)
 		)
 		(stroke
@@
 	(wire
 		(pts
-			(xy 76.2 97.79) (xy 91.44 97.79)
-		)
-		(stroke
-			(width 0)
-			(type default)
-		)
-	)
-	(wire
-		(pts
-			(xy 91.44 97.79) (xy 91.44 95.25)
+			(xy 87.63 97.79) (xy 105.41 97.79)
 		)
 		(stroke
@@
 	(wire
 		(pts
-			(xy 76.2 87.63) (xy 76.2 85.09)
+			(xy 87.63 87.63) (xy 87.63 85.09)
 		)
 		(stroke
@@
 	(wire
 		(pts
-			(xy 76.2 85.09) (xy 91.44 85.09)
-		)
-		(stroke
-			(width 0)
-			(type default)
-		)
-	)
-	(wire
-		(pts
 			(xy 115.57 97.79) (xy 129.54 97.79)
 		)
@@
 	(wire
 		(pts
-			(xy 91.44 85.09) (xy 91.44 87.63)
-		)
-		(stroke
-			(width 0)
-			(type default)
-		)
-	)
-	(wire
-		(pts
 			(xy 113.03 85.09) (xy 115.57 85.09)
 		)
@@
 	(wire
 		(pts
-			(xy 91.44 97.79) (xy 105.41 97.79)
-		)
-		(stroke
-			(width 0)
-			(type default)
-		)
-	)
-	(wire
-		(pts
 			(xy 115.57 85.09) (xy 129.54 85.09)
 		)
@@
 	(wire
 		(pts
-			(xy 76.2 95.25) (xy 76.2 97.79)
+			(xy 87.63 95.25) (xy 87.63 97.79)
 		)
 		(stroke
@@
 	(hierarchical_label "USB_5V"
 		(shape output)
-		(at 67.31 85.09 180)
+		(at 78.74 85.09 180)
 		(effects
 			(font
@@
 		(dnp no)
 		(fields_autoplaced yes)
-		(property "Reference" "C304"
+		(property "Reference" "C303"
 			(at 133.35 90.1699 0)
 			(effects
@@
 			(project "NosClock"
 				(path "/5a46aee9-b968-477e-a4a1-4edba06163a3/8ef51682-6928-4447-b545-210fc96c162e"
-					(reference "C304")
+					(reference "C303")
 					(unit 1)
 				)
@@
 		(dnp no)
 		(fields_autoplaced yes)
-		(property "Reference" "C303"
+		(property "Reference" "C302"
 			(at 119.38 90.1699 0)
 			(effects
@@
 			(project "NosClock"
 				(path "/5a46aee9-b968-477e-a4a1-4edba06163a3/8ef51682-6928-4447-b545-210fc96c162e"
-					(reference "C303")
+					(reference "C302")
 					(unit 1)
 				)
@@
 	(symbol
 		(lib_id "Device:C")
-		(at 91.44 91.44 0)
-		(unit 1)
-		(exclude_from_sim no)
-		(in_bom yes)
-		(on_board yes)
-		(dnp no)
-		(fields_autoplaced yes)
-		(property "Reference" "C302"
-			(at 95.25 90.1699 0)
-			(effects
-				(font
-					(size 1.27 1.27)
-				)
-				(justify left)
-			)
-		)
-		(property "Value" "10uF"
-			(at 95.25 92.7099 0)
-			(effects
-				(font
-					(size 1.27 1.27)
-				)
-				(justify left)
-			)
-		)
-		(property "Footprint" "Capacitor_SMD:C_0805_2012Metric"
-			(at 92.4052 95.25 0)
-			(effects
-				(font
-					(size 1.27 1.27)
-				)
-				(hide yes)
-			)
-		)
-		(property "Datasheet" "~"
-			(at 91.44 91.44 0)
-			(effects
-				(font
-					(size 1.27 1.27)
-				)
-				(hide yes)
-			)
-		)
-		(property "Description" "Unpolarized capacitor"
-			(at 91.44 91.44 0)
-			(effects
-				(font
-					(size 1.27 1.27)
-				)
-				(hide yes)
-			)
-		)
-		(property "Availability" ""
-			(at 91.44 91.44 0)
-			(effects
-				(font
-					(size 1.27 1.27)
-				)
-				(hide yes)
-			)
-		)
-		(property "Check_prices" ""
-			(at 91.44 91.44 0)
-			(effects
-				(font
-					(size 1.27 1.27)
-				)
-				(hide yes)
-			)
-		)
-		(property "Description_1" ""
-			(at 91.44 91.44 0)
-			(effects
-				(font
-					(size 1.27 1.27)
-				)
-				(hide yes)
-			)
-		)
-		(property "MF" ""
-			(at 91.44 91.44 0)
-			(effects
-				(font
-					(size 1.27 1.27)
-				)
-				(hide yes)
-			)
-		)
-		(property "MP" ""
-			(at 91.44 91.44 0)
-			(effects
-				(font
-					(size 1.27 1.27)
-				)
-				(hide yes)
-			)
-		)
-		(property "PARTNO" ""
-			(at 91.44 91.44 0)
-			(effects
-				(font
-					(size 1.27 1.27)
-				)
-				(hide yes)
-			)
-		)
-		(property "Package" ""
-			(at 91.44 91.44 0)
-			(effects
-				(font
-					(size 1.27 1.27)
-				)
-				(hide yes)
-			)
-		)
-		(property "Price" ""
-			(at 91.44 91.44 0)
-			(effects
-				(font
-					(size 1.27 1.27)
-				)
-				(hide yes)
-			)
-		)
-		(property "SnapEDA_Link" ""
-			(at 91.44 91.44 0)
-			(effects
-				(font
-					(size 1.27 1.27)
-				)
-				(hide yes)
-			)
-		)
-		(pin "1"
-		)
-		(pin "2"
-		)
-		(instances
-			(project "NosClock"
-				(path "/5a46aee9-b968-477e-a4a1-4edba06163a3/8ef51682-6928-4447-b545-210fc96c162e"
-					(reference "C302")
-					(unit 1)
-				)
-			)
-		)
-	)
-	(symbol
-		(lib_id "Device:C")
-		(at 76.2 91.44 0)
+		(at 87.63 91.44 0)
 		(unit 1)
 		(exclude_from_sim no)
@@
 		(fields_autoplaced yes)
 		(property "Reference" "C301"
-			(at 80.01 90.1699 0)
+			(at 91.44 90.1699 0)
 			(effects
 				(font
@@
 		)
 		(property "Value" "100nF"
-			(at 80.01 92.7099 0)
+			(at 91.44 92.7099 0)
 			(effects
 				(font
@@
 		)
 		(property "Footprint" "Capacitor_SMD:C_0603_1608Metric"
-			(at 77.1652 95.25 0)
+			(at 88.5952 95.25 0)
 			(effects
 				(font
@@
 		)
 		(property "Datasheet" "~"
-			(at 76.2 91.44 0)
+			(at 87.63 91.44 0)
 			(effects
 				(font
@@
 		)
 		(property "Description" "Unpolarized capacitor"
-			(at 76.2 91.44 0)
+			(at 87.63 91.44 0)
 			(effects
 				(font
@@
 		)
 		(property "Availability" ""
-			(at 76.2 91.44 0)
+			(at 87.63 91.44 0)
 			(effects
 				(font
@@
 		)
 		(property "Check_prices" ""
-			(at 76.2 91.44 0)
+			(at 87.63 91.44 0)
 			(effects
 				(font
@@
 		)
 		(property "Description_1" ""
-			(at 76.2 91.44 0)
+			(at 87.63 91.44 0)
 			(effects
 				(font
@@
 		)
 		(property "MF" ""
-			(at 76.2 91.44 0)
+			(at 87.63 91.44 0)
 			(effects
 				(font
@@
 		)
 		(property "MP" ""
-			(at 76.2 91.44 0)
+			(at 87.63 91.44 0)
 			(effects
 				(font
@@
 		)
 		(property "PARTNO" ""
-			(at 76.2 91.44 0)
+			(at 87.63 91.44 0)
 			(effects
 				(font
@@
 		)
 		(property "Package" ""
-			(at 76.2 91.44 0)
+			(at 87.63 91.44 0)
 			(effects
 				(font
@@
 		)
 		(property "Price" ""
-			(at 76.2 91.44 0)
+			(at 87.63 91.44 0)
 			(effects
 				(font
@@
 		)
 		(property "SnapEDA_Link" ""
-			(at 76.2 91.44 0)
-			(effects
-				(font
+			(at 87.63 91.44 0)
+			(effects
+				(font
