File: hardware/SK6812.kicad_sch (KiCad schematic)
At the start: 7 parts

Commit message: Static version (incomplete)
Parts:
- C302: footprint Capacitor_SMD:C_1206_3216Metric_Pad1.33x1.80mm_HandSolder -> Capacitor_SMD:C_0603_1608Metric
Changed lines of the file:
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@@
 		(dnp no)
 		(fields_autoplaced yes)
-		(property "Reference" "#PWR0304"
+		(property "Reference" "#PWR?"
 			(at 125.73 91.44 0)
 			(effects
@@
 				)
 			)
+			(project "SK6812"
+				(path "/d3b49bbc-89fa-4807-b130-f75fd2d42899"
+					(reference "#PWR?")
+					(unit 1)
+				)
+			)
 		)
 	)
@@
 		(dnp no)
 		(fields_autoplaced yes)
-		(property "Reference" "D301"
+		(property "Reference" "D?"
 			(at 62.23 67.31 0)
 			(effects
@@
 				)
 			)
+			(project "SK6812"
+				(path "/d3b49bbc-89fa-4807-b130-f75fd2d42899"
+					(reference "D?")
+					(unit 1)
+				)
+			)
 		)
 	)
@@
 		(dnp no)
 		(fields_autoplaced yes)
-		(property "Reference" "C301"
+		(property "Reference" "C?"
 			(at 72.39 82.1689 0)
 			(effects
@@
 				)
 			)
+			(project "SK6812"
+				(path "/d3b49bbc-89fa-4807-b130-f75fd2d42899"
+					(reference "C?")
+					(unit 1)
+				)
+			)
 		)
 	)
@@
 		(dnp no)
 		(fields_autoplaced yes)
-		(property "Reference" "C303"
+		(property "Reference" "C?"
 			(at 129.54 80.0099 0)
 			(effects
@@
 				)
 			)
+			(project "SK6812"
+				(path "/d3b49bbc-89fa-4807-b130-f75fd2d42899"
+					(reference "C?")
+					(unit 1)
+				)
+			)
 		)
 	)
@@
 		(dnp no)
 		(fields_autoplaced yes)
-		(property "Reference" "D302"
+		(property "Reference" "D?"
 			(at 113.03 95.1798 0)
 			(effects
@@
 				)
 			)
+			(project "SK6812"
+				(path "/d3b49bbc-89fa-4807-b130-f75fd2d42899"
+					(reference "D?")
+					(unit 1)
+				)
+			)
 		)
 	)
@@
 		(dnp no)
 		(fields_autoplaced yes)
-		(property "Reference" "#PWR0303"
+		(property "Reference" "#PWR?"
 			(at 100.33 115.57 0)
 			(effects
@@
 				)
 			)
+			(project "SK6812"
+				(path "/d3b49bbc-89fa-4807-b130-f75fd2d42899"
+					(reference "#PWR?")
+					(unit 1)
+				)
+			)
 		)
 	)
@@
 		(dnp no)
 		(fields_autoplaced yes)
-		(property "Reference" "#PWR0305"
+		(property "Reference" "#PWR?"
 			(at 147.32 115.57 0)
 			(effects
@@
 				)
 			)
+			(project "SK6812"
+				(path "/d3b49bbc-89fa-4807-b130-f75fd2d42899"
+					(reference "#PWR?")
+					(unit 1)
+				)
+			)
 		)
 	)
@@
 		(dnp no)
 		(fields_autoplaced yes)
-		(property "Reference" "#PWR0302"
+		(property "Reference" "#PWR?"
 			(at 87.63 92.71 0)
 			(effects
@@
 				)
 			)
+			(project "SK6812"
+				(path "/d3b49bbc-89fa-4807-b130-f75fd2d42899"
+					(reference "#PWR?")
+					(unit 1)
+				)
+			)
 		)
 	)
@@
 		(dnp no)
 		(fields_autoplaced yes)
-		(property "Reference" "R301"
+		(property "Reference" "R?"
 			(at 63.5 95.25 90)
 			(effects
@@
 				)
 			)
+			(project "SK6812"
+				(path "/d3b49bbc-89fa-4807-b130-f75fd2d42899"
+					(reference "R?")
+					(unit 1)
+				)
+			)
 		)
 	)
@@
 		(dnp no)
 		(fields_autoplaced yes)
-		(property "Reference" "#PWR0301"
+		(property "Reference" "#PWR?"
 			(at 68.58 92.71 0)
 			(effects
@@
 				)
 			)
+			(project "SK6812"
+				(path "/d3b49bbc-89fa-4807-b130-f75fd2d42899"
+					(reference "#PWR?")
+					(unit 1)
+				)
+			)
 		)
 	)
@@
 		(dnp no)
 		(fields_autoplaced yes)
-		(property "Reference" "C302"
+		(property "Reference" "C?"
 			(at 91.44 81.2799 0)
 			(effects
@@
 			)
 		)
-		(property "Footprint" "Capacitor_SMD:C_1206_3216Metric_Pad1.33x1.80mm_HandSolder"
+		(property "Footprint" "Capacitor_SMD:C_0603_1608Metric"
 			(at 88.5952 86.36 0)
 			(effects
@@
 				)
 			)
+			(project "SK6812"
+				(path "/d3b49bbc-89fa-4807-b130-f75fd2d42899"
+					(reference "C?")
+					(unit 1)
+				)
+			)
 		)
 	)
@@
 		(dnp no)
 		(fields_autoplaced yes)
-		(property "Reference" "D303"
+		(property "Reference" "D?"
 			(at 160.02 95.1798 0)
 			(effects
@@
 				)
 			)
-		)
-	)
+			(project "SK6812"
+				(path "/d3b49bbc-89fa-4807-b130-f75fd2d42899"
+					(reference "D?")
+					(unit 1)
+				)
+			)
+		)
+	)
+	(sheet_instances
+		(path "/"
+			(page "1")
+		)
+	)
+	(embedded_fonts no)
 )
