File: hardware/_autosave-Colon.kicad_sch (KiCad schematic)
At the start: 5 parts, among them Q902 MMBTA42

Commit message: 2/static version
Parts:
- added N801: INS-1, mynixies:mynixies-INS-1, symbol mynixies:INS-1
- added R801: 330K, Resistor_SMD:R_1206_3216Metric, symbol Device:R
- renumbered N903 to N1401, Q902 to Q1401, R902 to R1401, R906 to R1402, R912 to R1403
Connections:
- net +170V: now also N801.P$2 (A)
- net at Q1401.3 (C), R1403.1: now also R801.1
- new net: N801.P$1 (C), R801.2
Other:
- moved on the sheet: N1401, R1403
