File: hardware/HighSideSwitch.kicad_sch (KiCad schematic)
At the start: 5 parts, among them Q901 MMBTA42

Commit message: 2/static version
Parts:
- removed N902: INS-1, mynixies:mynixies-INS-1, symbol mynixies:INS-1
- removed Q901: MMBTA42, Package_TO_SOT_SMD:SOT-23, symbol Transistor_BJT:MMBTA42
- removed R903: 10K, Resistor_SMD:R_0603_1608Metric, symbol Device:R
- removed R908: 47K, Resistor_SMD:R_0603_1608Metric, symbol Device:R
- removed R911: 330K, Resistor_SMD:R_1206_3216Metric, symbol Device:R
- added Q701: MPSA92, Package_TO_SOT_THT:TO-92_Inline, symbol Transistor_BJT:MPSA92
- added Q702: MPSA42, Package_TO_SOT_THT:TO-92_Inline, symbol Transistor_BJT:MPSA42
- added R701, R702: 220K, Resistor_SMD:R_1206_3216Metric, symbol Device:R
- added R703: 10K, Resistor_SMD:R_0603_1608Metric, symbol Device:R
- added R704: 47K, Resistor_SMD:R_0603_1608Metric, symbol Device:R
Connections:
- net EN: now also R703.1
- net GND: now also Q702.1 (E), R704.1
- new net: Q701.2 (B), R701.2, R702.2
- new net: Q702.3 (C), R702.1
- new net: Q702.2 (B), R703.2, R704.2
- new net VIN: Q701.1 (E), R701.1
- new net VOUT: Q701.3 (C)

Commit message: Finalize schematics
Parts:
- removed Q701: MPSA92, Package_TO_SOT_THT:TO-92_Inline, symbol Transistor_BJT:MPSA92
- removed Q702: MPSA42, Package_TO_SOT_THT:TO-92_Inline, symbol Transistor_BJT:MPSA42
- added Q701: MMBTA92, Package_TO_SOT_SMD:SOT-23, symbol Transistor_BJT:MMBTA92
- added Q702: MMBTA42, Package_TO_SOT_SMD:SOT-23, symbol Transistor_BJT:MMBTA42
Connections:
- net GND: now also Q702.2 (E)
- net VIN: now also Q701.2 (E)
- net VOUT: now also Q701.3 (C)
- net at R701.2, R702.2: now also Q701.1 (B)
- net at R702.1: now also Q702.3 (C)
- net at R703.2, R704.2: now also Q702.1 (B)
Changed lines of the file:
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@@
-	)
-	(symbol
-		(lib_id "Transistor_BJT:MPSA92")
-		(at 148.59 90.17 0)
-		(mirror x)
-		(unit 1)
-		(exclude_from_sim no)
-		(in_bom yes)
-		(on_board yes)
-		(dnp no)
-		(property "Reference" "Q701"
-			(at 153.67 91.4401 0)
-			(effects
-				(font
-					(size 1.27 1.27)
-				)
-				(justify left)
-			)
-		)
-		(property "Value" "MPSA92"
-			(at 153.67 88.9001 0)
-			(effects
-				(font
-					(size 1.27 1.27)
-				)
-				(justify left)
-			)
-		)
-		(property "Footprint" "Package_TO_SOT_THT:TO-92_Inline"
-			(at 153.67 88.265 0)
-			(effects
-				(font
-					(size 1.27 1.27)
-					(italic yes)
-				)
-				(justify left)
-				(hide yes)
-			)
-		)
-		(property "Datasheet" "http://www.onsemi.com/pub_link/Collateral/MPSA92-D.PDF"
-			(at 148.59 90.17 0)
-			(effects
-				(font
-					(size 1.27 1.27)
-				)
-				(justify left)
-				(hide yes)
-			)
-		)
-		(property "Description" "0.5A Ic, 300V Vce, PNP High Voltage Transistor, TO-92"
-			(at 148.59 90.17 0)
-			(effects
-				(font
-					(size 1.27 1.27)
-				)
-				(hide yes)
-			)
-		)
-		(pin "2"
-		)
-		(pin "3"
-		)
-		(pin "1"
-		)
-		(instances
-			(project "NosClock"
-				(path "/5a46aee9-b968-477e-a4a1-4edba06163a3/cbfce168-24b0-4ff9-a45f-71f9f499ca5c/1c424bc5-98a3-4407-a843-d84953973710"
-					(reference "Q801")
-					(unit 1)
-				)
-				(path "/5a46aee9-b968-477e-a4a1-4edba06163a3/cbfce168-24b0-4ff9-a45f-71f9f499ca5c/39d58b35-aa77-439d-973f-4d49f0632d56"
-					(reference "Q901")
-					(unit 1)
-				)
-				(path "/5a46aee9-b968-477e-a4a1-4edba06163a3/cbfce168-24b0-4ff9-a45f-71f9f499ca5c/99ba67ee-e3d0-4e0a-b740-4da2fce5691d"
-					(reference "Q701")
-					(unit 1)
-				)
-			)
-		)
 	)
 	(symbol
@@
 	)
 	(symbol
-		(lib_id "Transistor_BJT:MPSA42")
+		(lib_id "Transistor_BJT:MMBTA42")
 		(at 123.19 102.87 0)
 		(unit 1)
@@
 			)
 		)
-		(property "Value" "MPSA42"
+		(property "Value" "MMBTA42"
 			(at 128.27 104.1399 0)
 			(effects
@@
 			)
 		)
-		(property "Footprint" "Package_TO_SOT_THT:TO-92_Inline"
+		(property "Footprint" "Package_TO_SOT_SMD:SOT-23"
 			(at 128.27 104.775 0)
 			(effects
@@
 			)
 		)
-		(property "Datasheet" "http://www.onsemi.com/pub_link/Collateral/MPSA42-D.PDF"
+		(property "Datasheet" "https://www.onsemi.com/pub/Collateral/MMBTA42LT1-D.PDF"
 			(at 123.19 102.87 0)
 			(effects
@@
 			)
 		)
-		(property "Description" "0.5A Ic, 300V Vce, NPN High Voltage Transistor, TO-92"
+		(property "Description" "0.5A Ic, 300V Vce, NPN High Voltage Transistor, SOT-23"
 			(at 123.19 102.87 0)
 			(effects
@@
 			)
 		)
+		(pin "3"
+		)
+		(pin "1"
+		)
 		(pin "2"
 		)
-		(pin "3"
-		)
-		(pin "1"
-		)
 		(instances
-			(project "NosClock"
+			(project ""
 				(path "/5a46aee9-b968-477e-a4a1-4edba06163a3/cbfce168-24b0-4ff9-a45f-71f9f499ca5c/1c424bc5-98a3-4407-a843-d84953973710"
 					(reference "Q802")
@@
 					(unit 1)
 				)
+			)
+		)
+	)
+	(symbol
+		(lib_id "Transistor_BJT:MMBTA92")
+		(at 148.59 90.17 0)
+		(mirror x)
+		(unit 1)
+		(exclude_from_sim no)
+		(in_bom yes)
+		(on_board yes)
+		(dnp no)
+		(property "Reference" "Q701"
+			(at 153.67 91.4401 0)
+			(effects
+				(font
+					(size 1.27 1.27)
+				)
+				(justify left)
+			)
+		)
+		(property "Value" "MMBTA92"
+			(at 153.67 88.9001 0)
+			(effects
+				(font
+					(size 1.27 1.27)
+				)
+				(justify left)
+			)
+		)
+		(property "Footprint" "Package_TO_SOT_SMD:SOT-23"
+			(at 153.67 88.265 0)
+			(effects
+				(font
+					(size 1.27 1.27)
+					(italic yes)
+				)
+				(justify left)
+				(hide yes)
+			)
+		)
+		(property "Datasheet" "https://www.onsemi.com/pub/Collateral/MMBTA92LT1-D.PDF"
+			(at 148.59 90.17 0)
+			(effects
+				(font
+					(size 1.27 1.27)
+				)
+				(justify left)
+				(hide yes)
+			)
+		)
+		(property "Description" "0.5A Ic, 300V Vce, PNP High Voltage Transistor, SOT-23"
+			(at 148.59 90.17 0)
+			(effects
+				(font
+					(size 1.27 1.27)
+				)
+				(hide yes)
+			)
+		)
+		(pin "1"
+		)
+		(pin "3"
+		)
+		(pin "2"
+		)
+		(instances
+			(project ""
+				(path "/5a46aee9-b968-477e-a4a1-4edba06163a3/cbfce168-24b0-4ff9-a45f-71f9f499ca5c/1c424bc5-98a3-4407-a843-d84953973710"
+					(reference "Q801")
+					(unit 1)
+				)
+				(path "/5a46aee9-b968-477e-a4a1-4edba06163a3/cbfce168-24b0-4ff9-a45f-71f9f499ca5c/39d58b35-aa77-439d-973f-4d49f0632d56"
+					(reference "Q901")
+					(unit 1)
+				)
+				(path "/5a46aee9-b968-477e-a4a1-4edba06163a3/cbfce168-24b0-4ff9-a45f-71f9f499ca5c/99ba67ee-e3d0-4e0a-b740-4da2fce5691d"
+					(reference "Q701")
+					(unit 1)
+				)
