File: hardware/NosClock.kicad_pcb (KiCad board)
At the start: 2 copper layers, 17 parts, among them Q201 MPSA92, Q202 P4NK60ZFP, U201 MC34063AP

Commit message: MAX1771
Parts:
- removed C201: 100nF, Capacitor_THT:C_Disc_D5.0mm_W2.5mm_P2.50mm
- removed C202: 220uF, Capacitor_THT:CP_Radial_D8.0mm_P3.80mm
- removed C203, C205: 1nF, Capacitor_THT:C_Disc_D5.0mm_W2.5mm_P2.50mm
- removed C204: 2.2uF 400v, Capacitor_THT:CP_Radial_D13.0mm_P5.00mm
- removed D201, D202: HER108, Diode_THT:D_DO-41_SOD81_P10.16mm_Horizontal
- removed L201: 150uH, Inductor_SMD:L_Bourns_SRR1260
- removed Q201: MPSA92, Package_TO_SOT_THT:TO-92_Inline
- removed Q202: P4NK60ZFP, Package_TO_SOT_THT:TO-220-3_Vertical
- removed R201: 0.1R, Resistor_THT:R_Axial_DIN0207_L6.3mm_D2.5mm_P10.16mm_Horizontal
- removed R202: 10K, Resistor_THT:R_Axial_DIN0207_L6.3mm_D2.5mm_P10.16mm_Horizontal
- removed R203: 1K, Resistor_THT:R_Axial_DIN0207_L6.3mm_D2.5mm_P10.16mm_Horizontal
- removed R204: 1M, Resistor_THT:R_Axial_DIN0207_L6.3mm_D2.5mm_P10.16mm_Horizontal
- removed R205: 330K, Resistor_THT:R_Axial_DIN0207_L6.3mm_D2.5mm_P10.16mm_Horizontal
- removed U201: MC34063AP, Package_DIP:DIP-8_W7.62mm
- removed VR201: P160KN-0QC15B500K, NosLib:P160
- added C103: 100uF 10V, Capacitor_THT:CP_Radial_D6.3mm_P2.50mm, B.Cu at (28.8, 151.1)
- added C302: 100nF, Capacitor_SMD:C_1206_3216Metric_Pad1.33x1.80mm_HandSolder, F.Cu at (36.1, 174.4)
- added C303: 100nF, Capacitor_SMD:C_1206_3216Metric_Pad1.33x1.80mm_HandSolder, F.Cu at (44.1, 174.4)
- added C304: 100nF, Capacitor_SMD:C_1206_3216Metric_Pad1.33x1.80mm_HandSolder, F.Cu at (60.0, 171.4)
- added C305: 10uF 400V (4.7uF 250V), Capacitor_THT:CP_Radial_D10.0mm_P5.00mm, B.Cu at (69.0, 170.0)
- added C306: 100nF 250V, Capacitor_SMD:C_1206_3216Metric_Pad1.33x1.80mm_HandSolder, F.Cu at (71.6, 165.0)
- added C307: 10uF 25V, Capacitor_SMD:C_1206_3216Metric_Pad1.33x1.80mm_HandSolder, F.Cu at (40.1, 174.4)
- added D301: UF4007 (ES2J), Diode_THT:D_DO-41_SOD81_P7.62mm_Horizontal, B.Cu at (57.8, 154.4)
- added L301: 100uH, Inductor_SMD:L_10.4x10.4_H4.8, F.Cu at (33.3, 165.4)
- added NT301: NetTie_2, NetTie:NetTie-2_SMD_Pad0.5mm, F.Cu at (37.2, 172.9)
- added NT303: NetTie_2, NetTie:NetTie-2_SMD_Pad0.5mm, F.Cu at (50.0, 160.4)
- added NX101: ~, nixies-us:nixies-us-IN-12-DSUB, B.Cu at (38.5, 133.7)
- added Q301: IRF740 (FQD12N20L), Package_TO_SOT_THT:TO-220-3_Vertical, B.Cu at (45.4, 159.4)
- added R101: 10K, Resistor_SMD:R_2512_6332Metric_Pad1.40x3.35mm_HandSolder, F.Cu at (61.8, 149.4)
- added R301: 0.1R, Resistor_SMD:R_2512_6332Metric_Pad1.40x3.35mm_HandSolder, F.Cu at (60.0, 163.4)
- added R302: 910K, Resistor_SMD:R_1206_3216Metric_Pad1.30x1.75mm_HandSolder, F.Cu at (55.0, 176.4)
- added R303: 16K, Resistor_SMD:R_0805_2012Metric_Pad1.20x1.40mm_HandSolder, F.Cu at (55.0, 180.4)
- added R304: 910K, Resistor_SMD:R_1206_3216Metric_Pad1.30x1.75mm_HandSolder, F.Cu at (61.0, 176.4)
- added TP101: A, TestPoint:TestPoint_Pad_3.0x3.0mm, F.Cu at (68.8, 122.0)
- added TP102: B, TestPoint:TestPoint_Pad_3.0x3.0mm, F.Cu at (68.8, 140.0)
- added TP103: C, TestPoint:TestPoint_Pad_3.0x3.0mm, F.Cu at (68.8, 146.0)
- added TP104: D, TestPoint:TestPoint_Pad_3.0x3.0mm, F.Cu at (68.8, 128.0)
- added TP105: 5V, TestPoint:TestPoint_Pad_3.0x3.0mm, F.Cu at (68.8, 134.0)
- added TP301: 12V, TestPoint:TestPoint_Pad_3.0x3.0mm, F.Cu at (31.0, 180.4)
- added TP302: PWR_GND, TestPoint:TestPoint_Pad_3.0x3.0mm, F.Cu at (37.0, 180.4)
- added TP303: PWR_GND, TestPoint:TestPoint_Pad_3.0x3.0mm, F.Cu at (68.8, 158.0)
- added TP304: 170V, TestPoint:TestPoint_Pad_3.0x3.0mm, F.Cu at (68.8, 152.0)
- added TP305: PWM, TestPoint:TestPoint_Pad_3.0x3.0mm, F.Cu at (48.0, 180.4)
- added U101: К155ИД1, Package_DIP:DIP-16_W7.62mm, B.Cu at (60.1, 125.8)
- added U102: AMS1117-5, Package_TO_SOT_SMD:SOT-223-3_TabPin2, F.Cu at (37.8, 153.8)
- added U301: MAX1771xSA, Package_SO:SO-8_3.9x4.9mm_P1.27mm, F.Cu at (51.0, 167.4)
Routing:
- net GND: track 0.00 -> 198.7 mm, vias 0 -> 2
- net 5V: track 0.00 -> 124.0 mm
- net Net-(U101-~{Q9}): track 0.00 -> 57.0 mm
- net /MAX1771/170V: track 0.00 -> 49.0 mm
- net Net-(U101-~{Q8}): track 0.00 -> 44.0 mm
- net 12V: track 0.00 -> 40.6 mm
- net Net-(U101-~{Q0}): track 0.00 -> 39.4 mm
- net Net-(U101-~{Q1}): track 0.00 -> 37.1 mm
- net Net-(U101-~{Q7}): track 0.00 -> 36.4 mm
- net Net-(U101-~{Q2}): track 0.00 -> 32.4 mm
- net Net-(NX101-PadA): track 0.00 -> 28.7 mm
- net /MAX1771/L_D: track 0.00 -> 24.1 mm
- net Net-(U101-~{Q6}): track 0.00 -> 21.0 mm
- net Net-(U301-FB): track 0.00 -> 16.0 mm
- net Net-(U301-V+): track 0.00 -> 14.8 mm
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Other:
- board outline added: 50 x 70 mm
- board text added: "Top"

Commit message: UC3843
Parts:
- removed C302, C303, C304: 100nF, Capacitor_SMD:C_1206_3216Metric_Pad1.33x1.80mm_HandSolder
- removed C305: 10uF 400V (4.7uF 250V), Capacitor_THT:CP_Radial_D10.0mm_P5.00mm
- removed C306: 100nF 250V, Capacitor_SMD:C_1206_3216Metric_Pad1.33x1.80mm_HandSolder
- removed C307: 10uF 25V, Capacitor_SMD:C_1206_3216Metric_Pad1.33x1.80mm_HandSolder
- removed D301: UF4007 (ES2J), Diode_THT:D_DO-41_SOD81_P7.62mm_Horizontal
- removed L301: 100uH, Inductor_SMD:L_10.4x10.4_H4.8
- removed NT301, NT303: NetTie_2, NetTie:NetTie-2_SMD_Pad0.5mm
- removed Q301: IRF740 (FQD12N20L), Package_TO_SOT_THT:TO-220-3_Vertical
- removed R301: 0.1R, Resistor_SMD:R_2512_6332Metric_Pad1.40x3.35mm_HandSolder
- removed R302, R304: 910K, Resistor_SMD:R_1206_3216Metric_Pad1.30x1.75mm_HandSolder
- removed R303: 16K, Resistor_SMD:R_0805_2012Metric_Pad1.20x1.40mm_HandSolder
- removed TP301: 12V, TestPoint:TestPoint_Pad_3.0x3.0mm
- removed TP302, TP303: PWR_GND, TestPoint:TestPoint_Pad_3.0x3.0mm
- removed TP304: 170V, TestPoint:TestPoint_Pad_3.0x3.0mm
- removed TP305: PWM, TestPoint:TestPoint_Pad_3.0x3.0mm
- removed U301: MAX1771xSA, Package_SO:SO-8_3.9x4.9mm_P1.27mm
- added C401: 100nF, Capacitor_SMD:C_1206_3216Metric_Pad1.33x1.80mm_HandSolder, F.Cu at (40.6, 184.3)
- added C402: 100pF, Capacitor_SMD:C_1206_3216Metric_Pad1.33x1.80mm_HandSolder, F.Cu at (25.6, 155.3)
- added C403: 1nF, Capacitor_SMD:C_1206_3216Metric_Pad1.33x1.80mm_HandSolder, F.Cu at (25.1, 171.3)
- added C404: 10uF 400V (4.7uF 250V), Capacitor_THT:CP_Radial_D10.0mm_P5.00mm, B.Cu at (56.0, 158.3)
- added D401: UF4007, Diode_THT:D_DO-41_SOD81_P7.62mm_Horizontal, F.Cu at (55.4, 167.3)
- added L401: 100uH, Inductor_SMD:L_APV_APH1030, F.Cu at (50.6, 178.3)
- added Q401: IRF740, Package_TO_SOT_THT:TO-220-3_Vertical, B.Cu at (37.5, 168.0)
- added R401: 150K, Resistor_SMD:R_1206_3216Metric_Pad1.30x1.75mm_HandSolder, F.Cu at (25.6, 160.3)
- added R402: 47K, Resistor_SMD:R_1206_3216Metric_Pad1.30x1.75mm_HandSolder, F.Cu at (25.1, 167.3)
- added R403: 10R, Resistor_SMD:R_1206_3216Metric_Pad1.30x1.75mm_HandSolder, F.Cu at (40.6, 176.3)
- added R404: 0.5R, Resistor_SMD:R_1206_3216Metric_Pad1.30x1.75mm_HandSolder, F.Cu at (42.6, 163.3)
- added R405: 680K, Resistor_SMD:R_1206_3216Metric_Pad1.30x1.75mm_HandSolder, F.Cu at (42.6, 155.3)
- added R406: 10K, Resistor_SMD:R_1206_3216Metric_Pad1.30x1.75mm_HandSolder, F.Cu at (42.6, 159.3)
- added TP104: GND, TestPoint:TestPoint_Pad_3.0x3.0mm, F.Cu at (64.4, 176.9)
- added TP107: 12V, TestPoint:TestPoint_Pad_3.0x3.0mm, F.Cu at (64.4, 182.9)
- added TP108: 170V, TestPoint:TestPoint_Pad_3.0x3.0mm, F.Cu at (64.4, 153.3)
- added U401: UC3843_SOIC8, Package_SO:SOIC-8_3.9x4.9mm_P1.27mm, F.Cu at (32.6, 178.3)
- moved C101 35.7 mm to (63.6, 159.3), turned to 180 degrees
- moved U101 29.3 mm to (62.6, 169.3)
- moved NX101 4.58 mm to (34.1, 135.0)
- moved U102 4.58 mm to (55.7, 127.1)
- moved R101 4.58 mm to (57.4, 150.7)
- moved TP101 4.58 mm to (64.4, 129.3)
- moved TP102 4.58 mm to (64.4, 135.3)
- moved TP103 4.58 mm to (64.4, 147.3)
- moved TP105 4.58 mm to (64.4, 141.3)
- moved TP106 4.58 mm to (64.4, 123.3)
- renumbered C103 to C101, TP104 to TP101, TP105 to TP102, TP102 to TP105, TP101 to TP106, U102 to U101, U101 to U102
Connections:
- R101 pad 2: /MAX1771/170V -> /UC3843/170V
Routing:
- net 5V: track 124.0 -> 45.7 mm
- net Net-(U401-FB): track 0.00 -> 49.5 mm
- net /MAX1771/170V: track 49.0 -> 0.00 mm
- net GND: track 198.7 -> 161.0 mm, vias 2 -> 0
- net /UC3843/170V: track 0.00 -> 36.7 mm
- net Net-(U401-VREF): track 0.00 -> 30.4 mm, vias 0 -> 2
- net Net-(Q401-S): track 0.00 -> 27.7 mm
- net /MAX1771/L_D: track 24.1 -> 0.00 mm
- net Net-(D401-A): track 0.00 -> 23.7 mm
- net Net-(U401-COMP): track 0.00 -> 23.6 mm
- net Net-(U301-FB): track 16.0 -> 0.00 mm
- net Net-(U301-V+): track 14.8 -> 0.00 mm
- net Net-(U401-RC): track 0.00 -> 11.3 mm
- net /MAX1771/PWM: track 11.3 -> 0.00 mm
- net Net-(U401-OUT): track 0.00 -> 10.5 mm
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
Commit message: Lamps & 3.3v/5v
Parts:
- removed NX101: ~, nixies-us:nixies-us-IN-12-DSUB
- removed TP101: D, TestPoint:TestPoint_Pad_3.0x3.0mm
- removed TP102: 5V, TestPoint:TestPoint_Pad_3.0x3.0mm
- removed TP103: C, TestPoint:TestPoint_Pad_3.0x3.0mm
- removed TP104: GND, TestPoint:TestPoint_Pad_3.0x3.0mm
- removed TP105: B, TestPoint:TestPoint_Pad_3.0x3.0mm
- removed TP106: A, TestPoint:TestPoint_Pad_3.0x3.0mm
- removed TP107: 12V, TestPoint:TestPoint_Pad_3.0x3.0mm
- removed TP108: 170V, TestPoint:TestPoint_Pad_3.0x3.0mm
- removed U101: AMS1117-5, Package_TO_SOT_SMD:SOT-223-3_TabPin2
- added C201: 10uF, Capacitor_SMD:C_0805_2012Metric_Pad1.18x1.45mm_HandSolder, F.Cu at (-42.6, 35.6)
- added C202: 10uF, Capacitor_SMD:C_0805_2012Metric_Pad1.18x1.45mm_HandSolder, F.Cu at (-42.6, 38.6)
- added C203: 100nF, Capacitor_SMD:C_0603_1608Metric_Pad1.08x0.95mm_HandSolder, F.Cu at (-47.2, 35.4)
- added C204: 3.9nF, Capacitor_SMD:C_0805_2012Metric_Pad1.18x1.45mm_HandSolder, F.Cu at (-42.6, 41.6)
- added C205: 10nF, Capacitor_SMD:C_0603_1608Metric_Pad1.08x0.95mm_HandSolder, F.Cu at (-47.2, 37.9)
- added C206: 22uF, Capacitor_SMD:C_0805_2012Metric_Pad1.18x1.45mm_HandSolder, F.Cu at (-42.6, 44.6)
- added C207: 22uF, Capacitor_SMD:C_0805_2012Metric_Pad1.18x1.45mm_HandSolder, F.Cu at (-42.6, 47.6)
- added C301: 100nF, Capacitor_SMD:C_0603_1608Metric_Pad1.08x0.95mm_HandSolder, F.Cu at (-42.4, 60.7)
- added C302: 10uF, Capacitor_SMD:C_0805_2012Metric_Pad1.18x1.45mm_HandSolder, F.Cu at (-47.0, 61.0)
- added C303: 100nF, Capacitor_SMD:C_0603_1608Metric_Pad1.08x0.95mm_HandSolder, F.Cu at (-42.4, 63.2)
- added C304: 10uF, Capacitor_SMD:C_0805_2012Metric_Pad1.18x1.45mm_HandSolder, F.Cu at (-47.0, 64.0)
- added D101: ES1J, Diode_SMD:D_SMA_Handsoldering, F.Cu at (-10.5, -3.00)
- added D501: SK6812MINI_ALI, LED_SMD:LED_SK6812MINI_PLCC4_3.5x3.5mm_P1.75mm, F.Cu at (264.2, 119.9)
- added D502: SK6812MINI_ALI, LED_SMD:LED_SK6812MINI_PLCC4_3.5x3.5mm_P1.75mm, F.Cu at (264.8, 130.9)
- added D503: SK6812MINI_ALI, LED_SMD:LED_SK6812MINI_PLCC4_3.5x3.5mm_P1.75mm, F.Cu at (289.0, 121.0)
- added D504: SK6812MINI_ALI, LED_SMD:LED_SK6812MINI_PLCC4_3.5x3.5mm_P1.75mm, F.Cu at (289.0, 131.0)
- added D601: SK6812MINI_ALI, LED_SMD:LED_SK6812MINI_PLCC4_3.5x3.5mm_P1.75mm, F.Cu at (253.7, 55.1)
- added D602: SK6812MINI_ALI, LED_SMD:LED_SK6812MINI_PLCC4_3.5x3.5mm_P1.75mm, F.Cu at (222.8, 55.1)
- added D603: SK6812MINI_ALI, LED_SMD:LED_SK6812MINI_PLCC4_3.5x3.5mm_P1.75mm, F.Cu at (253.7, 60.2)
- added D604: SK6812MINI_ALI, LED_SMD:LED_SK6812MINI_PLCC4_3.5x3.5mm_P1.75mm, F.Cu at (222.8, 60.2)
- added D701: SK6812MINI_ALI, LED_SMD:LED_SK6812MINI_PLCC4_3.5x3.5mm_P1.75mm, F.Cu at (192.0, 55.1)
- added D702: SK6812MINI_ALI, LED_SMD:LED_SK6812MINI_PLCC4_3.5x3.5mm_P1.75mm, F.Cu at (192.0, 89.2)
- added D703: SK6812MINI_ALI, LED_SMD:LED_SK6812MINI_PLCC4_3.5x3.5mm_P1.75mm, F.Cu at (192.0, 60.2)
- added D704: SK6812MINI_ALI, LED_SMD:LED_SK6812MINI_PLCC4_3.5x3.5mm_P1.75mm, F.Cu at (192.0, 94.3)
- added J101: USB_C_Receptacle_USB2.0_16P, Connector_USB:USB_C_Receptacle_HRO_TYPE-C-31-M-12, F.Cu at (57.1, 79.0)
- added J102: AC, NosLib:TerminalBlock_Phoenix_MKDS-1,5-2-5.08_1x02_P5.08mm_Horizontal, F.Cu at (-18.0, 9.00)
- added L201: 10uH 4A, Inductor_SMD:L_6.3x6.3_H3, F.Cu at (-35.9, 38.0)
- added NT101: NetTie_2, NetTie:NetTie-2_SMD_Pad0.5mm, F.Cu at (71.6, 77.0)
- added NT201: NetTie_IN_EN, NetTie:NetTie-2_SMD_Pad0.5mm, F.Cu at (-30.5, 42.7)
- added NT202: NetTie_GND, NetTie:NetTie-2_SMD_Pad0.5mm, F.Cu at (-30.5, 44.2)
- added NT203: NetTie_SW_BS, NetTie:NetTie-2_SMD_Pad0.5mm, F.Cu at (-30.5, 45.7)
- added NT204: NetTie_SW_FB, NetTie:NetTie-2_SMD_Pad0.5mm, F.Cu at (-30.5, 47.2)
- added NX501: IN-12B, nixies-us:nixies-us-IN-12, F.Cu at (264.8, 125.2)
- added NX502: IN-12B, nixies-us:nixies-us-IN-12, F.Cu at (287.4, 125.5)
- added NX601: IN-12B, nixies-us:nixies-us-IN-12, F.Cu at (210.9, 42.0)
- added NX602: IN-12B, nixies-us:nixies-us-IN-12, F.Cu at (241.8, 42.0)
- added NX701: IN-12B, nixies-us:nixies-us-IN-12, F.Cu at (174.0, 40.0)
- added NX702: IN-12B, nixies-us:nixies-us-IN-12, F.Cu at (180.0, 76.2)
- added R102: 10K, Resistor_SMD:R_0603_1608Metric_Pad0.98x0.95mm_HandSolder, F.Cu at (65.1, 77.0)
- added R103: 5.1K, Resistor_SMD:R_0603_1608Metric_Pad0.98x0.95mm_HandSolder, F.Cu at (65.1, 79.5)
- added R104: 5.1K, Resistor_SMD:R_0603_1608Metric_Pad0.98x0.95mm_HandSolder, F.Cu at (65.1, 82.0)
- added R201: 100K, Resistor_SMD:R_0603_1608Metric_Pad0.98x0.95mm_HandSolder, F.Cu at (-47.2, 40.4)
- added R202: 7.5K, Resistor_SMD:R_0603_1608Metric_Pad0.98x0.95mm_HandSolder, F.Cu at (-47.2, 42.9)
- added R203: 10K, Resistor_SMD:R_0603_1608Metric_Pad0.98x0.95mm_HandSolder, F.Cu at (-47.2, 45.4)
- added R204: 26.1K, Resistor_SMD:R_0603_1608Metric_Pad0.98x0.95mm_HandSolder, F.Cu at (-47.2, 47.9)
- added R501: 10K, Resistor_SMD:R_2512_6332Metric_Pad1.40x3.35mm_HandSolder, F.Cu at (258.0, 152.0)
- added R502: 10K, Resistor_SMD:R_2512_6332Metric_Pad1.40x3.35mm_HandSolder, F.Cu at (311.0, 153.0)
- added R601: 10K, Resistor_SMD:R_2512_6332Metric_Pad1.40x3.35mm_HandSolder, F.Cu at (205.9, 55.9)
- added R602: 10K, Resistor_SMD:R_2512_6332Metric_Pad1.40x3.35mm_HandSolder, F.Cu at (236.8, 55.9)
- added R701: 10K, Resistor_SMD:R_2512_6332Metric_Pad1.40x3.35mm_HandSolder, F.Cu at (175.1, 90.0)
- added R702: 10K, Resistor_SMD:R_2512_6332Metric_Pad1.40x3.35mm_HandSolder, F.Cu at (175.1, 55.9)
- added TP_101: BOOT, NosLib:TestPoint_Pad_1.0x1.0mm, F.Cu at (68.8, 74.7)
- added TP_102: EN, NosLib:TestPoint_Pad_1.0x1.0mm, F.Cu at (68.8, 77.8)
- added TP_103: GND, NosLib:TestPoint_Pad_1.0x1.0mm, F.Cu at (68.8, 80.8)
- added U201: MP2307DN-LF-Z, NosLib:SOIC-8-1EP_3.9x4.9mm_P1.27mm_EP2.29x3mm_ThermalVias, F.Cu at (-36.0, 45.3)
- added U301: AP7361-33ER-13, Package_TO_SOT_SMD:SOT-223-3_TabPin2, F.Cu at (-44.4, 55.4)
- added U501: 74HC595, Package_SO:TSSOP-16_4.4x5mm_P0.65mm, F.Cu at (278.0, 162.7)
- added U502: K155ID1, Package_DIP:DIP-16_W7.62mm, F.Cu at (278.1, 147.6)
- added U503: K155ID1, Package_DIP:DIP-16_W7.62mm, F.Cu at (255.5, 147.6)
- added U601: 74HC595, Package_SO:TSSOP-16_4.4x5mm_P0.65mm, F.Cu at (248.1, 102.1)
- added U602: K155ID1, Package_DIP:DIP-16_W7.62mm, F.Cu at (221.1, 32.7)
- added U603: K155ID1, Package_DIP:DIP-16_W7.62mm, F.Cu at (251.9, 32.7)
- added U701: 74HC595, Package_SO:TSSOP-16_4.4x5mm_P0.65mm, F.Cu at (226.0, 109.0)
- added U702: K155ID1, Package_DIP:DIP-16_W7.62mm, F.Cu at (190.2, 66.8)
- added U703: K155ID1, Package_DIP:DIP-16_W7.62mm, F.Cu at (190.2, 32.7)
- C101: value 100uF 10V -> 1uF; footprint Capacitor_THT:CP_Radial_D6.3mm_P2.50mm -> Capacitor_SMD:C_0805_2012Metric_Pad1.18x1.45mm_HandSolder; moved to F.Cu
- D401: value UF4007 -> ES1J; footprint Diode_THT:D_DO-41_SOD81_P7.62mm_Horizontal -> Diode_SMD:D_SMA_Handsoldering
- Q401: value IRF740 -> IRF740 (AOD11S60)
- R101: footprint Resistor_SMD:R_2512_6332Metric_Pad1.40x3.35mm_HandSolder -> Resistor_SMD:R_0603_1608Metric_Pad0.98x0.95mm_HandSolder
- U102: value К155ИД1 -> ESP32-C3-WROOM-02; footprint Package_DIP:DIP-16_W7.62mm -> PCM_Espressif:ESP32-C3-WROOM-02; moved to F.Cu
- moved C101 85.0 mm to (72.7, 74.7), turned to 0 degrees
- moved R101 76.6 mm to (65.1, 74.5)
- moved U102 62.0 mm to (61.5, 65.4), turned to 0 degrees
- moved C401 35.0 mm to (48.8, 150.3)
- moved C403 35.0 mm to (33.3, 137.3)
- moved D401 35.0 mm to (63.6, 133.3)
- moved L401 35.0 mm to (58.8, 144.3)
- moved Q401 35.0 mm to (45.7, 134.0)
- moved R402 35.0 mm to (33.3, 133.3)
- moved R403 35.0 mm to (48.8, 142.3)
- moved R404 35.0 mm to (50.8, 129.3)
- moved U401 35.0 mm to (40.8, 144.3)
- moved C402 35.0 mm to (33.8, 121.3)
- moved C404 35.0 mm to (64.2, 124.3)
- moved R401 35.0 mm to (33.8, 126.3)
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Connections:
- net 12V renamed +12V
- C101 pad 1: 5V -> EN
- R101 pad 1: Net-(NX101-PadA) -> BOOT
- R101 pad 2: /UC3843/170V -> GND
- U102 pad 1: Net-(U102-~{Q8}) -> unconnected-(U102-3V3-Pad1)
- U102 pad 10: Net-(U102-~{Q7}) -> CS
- U102 pad 11: Net-(U102-~{Q6}) -> unconnected-(U102-GPIO20/U0RXD-Pad11)
- U102 pad 12: GND -> unconnected-(U102-GPIO21/U0TXD-Pad12)
- U102 pad 13: Net-(U102-~{Q4}) -> USB_D-
- U102 pad 14: Net-(U102-~{Q5}) -> USB_D+
- U102 pad 15: Net-(U102-~{Q1}) -> ~{PWM}
- U102 pad 16: Net-(U102-~{Q0}) -> unconnected-(U102-GPIO2/ADC1_CH2-Pad16)
- U102 pad 2: Net-(U102-~{Q9}) -> EN
- U102 pad 3: Net-(U102-A) -> LED
- U102 pad 4: Net-(U102-D) -> unconnected-(U102-GPIO5/ADC2_CH0-Pad4)
- U102 pad 5: 5V -> SCK
- U102 pad 6: Net-(U102-B) -> MOSI
- U102 pad 7: Net-(U102-C) -> unconnected-(U102-GPIO8-Pad7)
- U102 pad 8: Net-(U102-~{Q2}) -> BOOT
- U102 pad 9: Net-(U102-~{Q3}) -> Net-(U102-GND-Pad19)
Routing:
- net GND: track 161.0 -> 0.00 mm
- net Net-(U102-~{Q9}): track 57.0 -> 0.00 mm
- net +12V: track 49.6 -> 0.00 mm
- net Net-(U401-FB): track 49.5 -> 0.00 mm
- net 5V: track 45.7 -> 0.00 mm
- net Net-(U102-~{Q8}): track 44.0 -> 0.00 mm
- net Net-(U102-~{Q0}): track 39.4 -> 0.00 mm
- net Net-(U102-~{Q1}): track 37.1 -> 0.00 mm
- net /UC3843/170V: track 36.7 -> 0.00 mm
- net Net-(U102-~{Q7}): track 36.4 -> 0.00 mm
- net Net-(U102-~{Q2}): track 32.4 -> 0.00 mm
- net Net-(U401-VREF): track 30.4 -> 0.00 mm, vias 2 -> 0
- net Net-(NX101-PadA): track 28.7 -> 0.00 mm
- net Net-(Q401-S): track 27.7 -> 0.00 mm
- net Net-(D401-A): track 23.7 -> 0.00 mm
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Other:
- board size 50 x 70 mm -> 309 x 88 mm

Commit message: Static version (incomplete)
Parts:
- removed C304: 10uF, Capacitor_SMD:C_0805_2012Metric_Pad1.18x1.45mm_HandSolder
- removed the D101 at (-10.5, -3.00)
- removed D502, D503, D504: SK6812MINI_ALI, LED_SMD:LED_SK6812MINI_PLCC4_3.5x3.5mm_P1.75mm
- removed NX501, NX502: IN-12B, nixies-us:nixies-us-IN-12
- removed R502: 10K, Resistor_SMD:R_2512_6332Metric_Pad1.40x3.35mm_HandSolder
- removed U501: 74HC595, Package_SO:TSSOP-16_4.4x5mm_P0.65mm
- removed U502, U503: K155ID1, Package_DIP:DIP-16_W7.62mm
- added C102: 100nF, Capacitor_SMD:C_0603_1608Metric, F.Cu at (62.6, 99.5)
- added C103: 100nF, Capacitor_SMD:C_0603_1608Metric, F.Cu at (112.6, 100.0)
- added C104: 100nF, Capacitor_SMD:C_0603_1608Metric, F.Cu at (76.7, 99.5)
- added C105: 100nF, Capacitor_SMD:C_0603_1608Metric, F.Cu at (126.7, 100.0)
- added C207: 100nF, Capacitor_SMD:C_0603_1608Metric, F.Cu at (92.5, 100.0)
- added C208: 100nF, Capacitor_SMD:C_0603_1608Metric, F.Cu at (42.5, 99.5)
- added C210: 100nF, Capacitor_SMD:C_0603_1608Metric, F.Cu at (56.6, 99.5)
- added C211: 100nF, Capacitor_SMD:C_0603_1608Metric, F.Cu at (106.6, 100.0)
- added C405: 4.7uF 250V, Capacitor_THT:CP_Radial_D8.0mm_P3.50mm, F.Cu at (220.7, 103.4)
- added C406: 220uF 35V, Capacitor_THT:CP_Radial_D6.3mm_P2.50mm, F.Cu at (206.0, 102.1)
- added C501: 100uF 10V, Capacitor_THT:CP_Radial_D6.3mm_P2.50mm, F.Cu at (82.5, 55.0)
- added C801: 100nF, Capacitor_SMD:C_0603_1608Metric, F.Cu at (162.6, 100.3)
- added C802: 100nF, Capacitor_SMD:C_0603_1608Metric, F.Cu at (142.5, 100.3)
- added C803: 100nF, Capacitor_SMD:C_0603_1608Metric, F.Cu at (176.7, 100.3)
- added C804: 100nF, Capacitor_SMD:C_0603_1608Metric, F.Cu at (156.6, 100.3)
- added D801: SK6812MINI_ALI, LED_SMD:LED_SK6812MINI_PLCC4_3.5x3.5mm_P1.75mm, F.Cu at (169.8, 105.9)
- added D802: SK6812MINI_ALI, LED_SMD:LED_SK6812MINI_PLCC4_3.5x3.5mm_P1.75mm, F.Cu at (149.2, 105.9)
- added D803: SK6812MINI_ALI, LED_SMD:LED_SK6812MINI_PLCC4_3.5x3.5mm_P1.75mm, F.Cu at (149.2, 115.9)
- added D804: SK6812MINI_ALI, LED_SMD:LED_SK6812MINI_PLCC4_3.5x3.5mm_P1.75mm, F.Cu at (169.8, 115.9)
- added N901: INS-1, mynixies:mynixies-INS-1, F.Cu at (84.6, 105.6)
- added N902: INS-1, mynixies:mynixies-INS-1, F.Cu at (84.6, 115.9)
- added N903: INS-1, mynixies:mynixies-INS-1, F.Cu at (134.6, 105.6)
- added N904: INS-1, mynixies:mynixies-INS-1, F.Cu at (134.6, 115.9)
- added NT102: NetTie_2, NetTie:NetTie-2_SMD_Pad0.5mm, F.Cu at (45.9, 174.7)
- added NT401: NetTie_2, NetTie:NetTie-2_SMD_Pad0.5mm, F.Cu at (207.3, 102.1)
- added NT402: NetTie_2, NetTie:NetTie-2_SMD_Pad0.5mm, F.Cu at (221.8, 108.8)
- added NT403: NetTie_2, NetTie:NetTie-2_SMD_Pad0.5mm, F.Cu at (227.1, 99.6)
- added NX801: IN-12B, nixies-us:nixies-us-IN-12, F.Cu at (170.1, 110.8)
- added NX802: IN-12B, nixies-us:nixies-us-IN-12, F.Cu at (150.0, 110.8)
- added Q901: MMBTA42, Package_TO_SOT_SMD:SOT-23, F.Cu at (84.6, 94.3)
- added Q902: MMBTA42, Package_TO_SOT_SMD:SOT-23, F.Cu at (134.6, 94.3)
- added Q903: MMBTA42, Package_TO_SOT_SMD:SOT-23, F.Cu at (137.4, 121.9)
- added Q904: MMBTA42, Package_TO_SOT_SMD:SOT-23, F.Cu at (87.4, 121.9)
- added R105: 4.7K, Resistor_SMD:R_0603_1608Metric, F.Cu at (98.8, 213.8)
- added R202: 22K, Resistor_SMD:R_2512_6332Metric, F.Cu at (46.6, 125.9)
- added R203: 22K, Resistor_SMD:R_2512_6332Metric, F.Cu at (96.6, 126.4)
- added R407: 10K, Resistor_SMD:R_0603_1608Metric, F.Cu at (228.6, 104.7)
- added R801: 10K, Resistor_SMD:R_0603_1608Metric, F.Cu at (165.1, 127.1)
- added R802: 22K, Resistor_SMD:R_2512_6332Metric, F.Cu at (172.6, 126.7)
- added R803: 22K, Resistor_SMD:R_2512_6332Metric, F.Cu at (146.6, 126.7)
- added R901: 10K, Resistor_SMD:R_0603_1608Metric, F.Cu at (24.3, 218.0)
- added R902: 10K, Resistor_SMD:R_0603_1608Metric, F.Cu at (134.6, 86.6)
- added R903: 10K, Resistor_SMD:R_0603_1608Metric, F.Cu at (84.6, 86.6)
- added R904: 10K, Resistor_SMD:R_0603_1608Metric, F.Cu at (81.4, 127.1)
- added R905: 10K, Resistor_SMD:R_0603_1608Metric, F.Cu at (131.4, 127.1)
- added R906: 47K, Resistor_SMD:R_0603_1608Metric, F.Cu at (134.6, 89.9)
- added R907: 47K, Resistor_SMD:R_0603_1608Metric, F.Cu at (87.4, 127.1)
- added R908: 47K, Resistor_SMD:R_0603_1608Metric, F.Cu at (84.6, 89.9)
- added R909: 47K, Resistor_SMD:R_0603_1608Metric, F.Cu at (137.4, 127.1)
- added R910: 330K, Resistor_SMD:R_1206_3216Metric, F.Cu at (81.4, 122.4)
- added R911: 330K, Resistor_SMD:R_1206_3216Metric, F.Cu at (84.6, 99.1)
- added R912: 330K, Resistor_SMD:R_1206_3216Metric, F.Cu at (134.6, 99.1)
- added R913: 330K, Resistor_SMD:R_1206_3216Metric, F.Cu at (131.4, 122.4)
- added U103: DS18B20, Package_TO_SOT_THT:TO-92_Inline, F.Cu at (98.7, 210.0)
- added U801: 74HC595, Package_SO:TSSOP-16_4.4x5mm_P0.65mm, F.Cu at (159.6, 124.8)
- added U802: K155ID1, Package_DIP:DIP-16_W7.62mm, F.Cu at (179.3, 87.3)
- added U803: K155ID1, Package_DIP:DIP-16_W7.62mm, F.Cu at (157.6, 87.3)
- added U901: 74HC595, Package_SO:TSSOP-16_4.4x5mm_P0.65mm, F.Cu at (19.3, 210.0)
- C101, C201, C202, C206: footprint Capacitor_SMD:C_0805_2012Metric_Pad1.18x1.45mm_HandSolder -> Capacitor_SMD:C_0805_2012Metric
- C203, C205, C301: footprint Capacitor_SMD:C_0603_1608Metric_Pad1.08x0.95mm_HandSolder -> Capacitor_SMD:C_0603_1608Metric
- C204: footprint Capacitor_SMD:C_0805_2012Metric_Pad1.18x1.45mm_HandSolder -> Capacitor_SMD:C_0603_1608Metric
- C209: renamed from C207; footprint Capacitor_SMD:C_0805_2012Metric_Pad1.18x1.45mm_HandSolder -> Capacitor_SMD:C_0805_2012Metric
- C302: value 10uF -> 100nF; footprint Capacitor_SMD:C_0805_2012Metric_Pad1.18x1.45mm_HandSolder -> Capacitor_SMD:C_0603_1608Metric
- C303: value 100nF -> 10uF; footprint Capacitor_SMD:C_0603_1608Metric_Pad1.08x0.95mm_HandSolder -> Capacitor_SMD:C_0805_2012Metric
- C401, C402, C403: footprint Capacitor_SMD:C_1206_3216Metric_Pad1.33x1.80mm_HandSolder -> Capacitor_SMD:C_0603_1608Metric
- C404: value 10uF 400V (4.7uF 250V) -> 1nF; footprint Capacitor_THT:CP_Radial_D10.0mm_P5.00mm -> Capacitor_SMD:C_0603_1608Metric; moved to F.Cu
- D401: footprint Diode_SMD:D_SMA_Handsoldering -> Diode_SMD:D_SMA
- D501: value SK6812MINI_ALI -> ES1J; footprint LED_SMD:LED_SK6812MINI_PLCC4_3.5x3.5mm_P1.75mm -> Diode_SMD:D_SMA_Handsoldering
- J101: value USB_C_Receptacle_USB2.0_16P -> AC; footprint Connector_USB:USB_C_Receptacle_HRO_TYPE-C-31-M-12 -> NosLib:TerminalBlock_Phoenix_MKDS-1,5-2-5.08_1x02_P5.08mm_Horizontal
- J102: value AC -> USB_C_Receptacle_USB2.0_16P; footprint NosLib:TerminalBlock_Phoenix_MKDS-1,5-2-5.08_1x02_P5.08mm_Horizontal -> Connector_USB:USB_C_Receptacle_HRO_TYPE-C-31-M-12
- Q401: value IRF740 (AOD11S60) -> AOD11S60; footprint Package_TO_SOT_THT:TO-220-3_Vertical -> Package_TO_SOT_SMD:TO-252-2; moved to F.Cu
- R101, R102, R103, R104, R201: footprint Resistor_SMD:R_0603_1608Metric_Pad0.98x0.95mm_HandSolder -> Resistor_SMD:R_0603_1608Metric
- R106: renamed from R702; value 10K -> 22K; footprint Resistor_SMD:R_2512_6332Metric_Pad1.40x3.35mm_HandSolder -> Resistor_SMD:R_2512_6332Metric
- R107: renamed from R602; value 10K -> 22K; footprint Resistor_SMD:R_2512_6332Metric_Pad1.40x3.35mm_HandSolder -> Resistor_SMD:R_2512_6332Metric
- R204: renamed from R202; footprint Resistor_SMD:R_0603_1608Metric_Pad0.98x0.95mm_HandSolder -> Resistor_SMD:R_0603_1608Metric
- R205: renamed from R203; value 10K -> 6.8K; footprint Resistor_SMD:R_0603_1608Metric_Pad0.98x0.95mm_HandSolder -> Resistor_SMD:R_0603_1608Metric
- R206: renamed from R204; value 26.1K -> 30K; footprint Resistor_SMD:R_0603_1608Metric_Pad0.98x0.95mm_HandSolder -> Resistor_SMD:R_0603_1608Metric
- R401, R402: footprint Resistor_SMD:R_1206_3216Metric_Pad1.30x1.75mm_HandSolder -> Resistor_SMD:R_0603_1608Metric
- R403: value 10R -> 1K; footprint Resistor_SMD:R_1206_3216Metric_Pad1.30x1.75mm_HandSolder -> Resistor_SMD:R_0603_1608Metric
- R404: value 0.5R -> 10R; footprint Resistor_SMD:R_1206_3216Metric_Pad1.30x1.75mm_HandSolder -> Resistor_SMD:R_0603_1608Metric
- R405: value 680K -> 0.5R; footprint Resistor_SMD:R_1206_3216Metric_Pad1.30x1.75mm_HandSolder -> Resistor_SMD:R_2512_6332Metric
- R406: value 10K -> 680K; footprint Resistor_SMD:R_1206_3216Metric_Pad1.30x1.75mm_HandSolder -> Resistor_SMD:R_1206_3216Metric
- R501: value 10K -> 330R; footprint Resistor_SMD:R_2512_6332Metric_Pad1.40x3.35mm_HandSolder -> Resistor_SMD:R_0603_1608Metric
- R601, R701: footprint Resistor_SMD:R_2512_6332Metric_Pad1.40x3.35mm_HandSolder -> Resistor_SMD:R_0603_1608Metric
- moved D204 211.8 mm to (49.2, 115.0)
- moved D202 210.6 mm to (49.2, 105.1)
- moved C403 206.7 mm to (238.7, 114.1), turned to 0 degrees
- moved R402 206.0 mm to (238.7, 117.3), turned to 0 degrees
- moved R401 201.8 mm to (234.3, 103.6)
- moved C402 201.6 mm to (234.3, 100.5)
- moved U401 198.9 mm to (236.5, 108.9), turned to 0 degrees
- moved C401 195.6 mm to (238.7, 103.7), turned to 180 degrees
- moved D501 194.6 mm to (77.5, 65.0)
- moved U601 189.8 mm to (59.6, 123.9), turned to -90 degrees
- moved R501 187.8 mm to (91.6, 65.0)
- moved R403 187.2 mm to (234.3, 117.3), turned to 180 degrees
- moved NX102 184.6 mm to (70.1, 110.0)
- moved U101 180.8 mm to (79.3, 86.5), turned to -90 degrees
- moved R406 179.5 mm to (228.6, 100.8)
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- renumbered D602 to D101, D702 to D102, D703 to D103, D604 to D104, D701 to D201, D601 to D202, D704 to D203, D603 to D204, NX702 to NX101, NX602 to NX102, NX701 to NX201, NX601 to NX202, U603 to U101, U702 to U102, U102 to U104, U703 to U201, U602 to U202, U201 to U203
Connections:
- net /TwoDigits2/74HC595_OUT renamed /Lamps/TwoDigits1/74HC595_OUT
- net /TwoDigits2/Digit1/SK6812MINI_OUT renamed /Lamps/TwoDigits1/Digit1/SK6812MINI_OUT
- net Net-(D401-A) renamed /UC3843/PWR_SW
- C302 pad 1: +5V -> +3V3
- C401 pad 1: +12V -> Net-(U401-VCC)
- C402 pad 2: Net-(U401-FB) -> /UC3843/FB
- C404 pad 1: /UC3843/170V -> Net-(U401-CS)
- D101 pad 1: /TwoDigits2/FIRST_SK6812MINI_VCC -> /Lamps/TwoDigits1/FIRST_SK6812MINI_VCC
- D101 pad 4: /TwoDigits1/SK_OUT -> /Lamps/TwoDigits1/SK_IN
- D102 pad 2: Net-(D702-DOUT) -> Net-(D102-DOUT)
- D102 pad 4: /TwoDigits3/Digit1/SK6812MINI_OUT -> /Lamps/TwoDigits1/SK_OUT
- D103 pad 2: /TwoDigits3/Digit1/SK6812MINI_OUT -> /Lamps/TwoDigits2/Digit1/SK6812MINI_OUT
- D103 pad 4: Net-(D701-DOUT) -> Net-(D102-DOUT)
- D201 pad 1: /TwoDigits3/FIRST_SK6812MINI_VCC -> +5V
- D201 pad 2: Net-(D701-DOUT) -> Net-(D201-DOUT)
- D201 pad 4: /TwoDigits2/SK_OUT -> /Lamps/TwoDigits2/Digit1/SK6812MINI_OUT
- D203 pad 2: /TwoDigits3/SK_OUT -> /Lamps/TwoDigits2/SK_OUT
- D203 pad 4: Net-(D702-DOUT) -> Net-(D201-DOUT)
- D204 pad 2: /TwoDigits2/SK_OUT -> /Lamps/TwoDigits1/SK_OUT
- D401 pad 1: /UC3843/170V -> +170V
- D501 pad 1: /TwoDigits1/FIRST_SK6812MINI_VCC -> /Lamps/TwoDigits1/FIRST_SK6812MINI_VCC
- D501 pad 2: Net-(D501-DOUT) -> +5V
- NT101 pad 1: Net-(J101-VBUS-PadA4) -> Net-(J102-VBUS-PadA4)
- NX101 pad A: Net-(NX702-PadA) -> Net-(NX101-PadA)
- NX201 pad A: Net-(NX701-PadA) -> Net-(NX201-PadA)
- NX202 pad A: Net-(NX601-PadA) -> Net-(NX202-PadA)
- Q401 pad 3: Net-(Q401-S) -> /UC3843/PWR_SEN
- R103 pad 1: Net-(J101-CC1) -> Net-(J102-CC1)
- R104 pad 1: Net-(J101-CC2) -> Net-(J102-CC2)
- R106 pad 1: Net-(NX701-PadA) -> Net-(NX101-PadA)
- R401 pad 2: Net-(U401-FB) -> /UC3843/FB
- R403 pad 1: Net-(U401-OUT) -> Net-(U401-CS)
- R403 pad 2: Net-(Q401-G) -> Net-(NT402-Pad2)
- R404 pad 1: Net-(Q401-S) -> Net-(U401-OUT)
- R404 pad 2: GND -> Net-(Q401-G)
- R405 pad 1: /UC3843/170V -> /UC3843/PWR_SEN
- R405 pad 2: Net-(U401-FB) -> /UC3843/PWR_GND
- R406 pad 1: Net-(U401-FB) -> Net-(NT403-Pad2)
- R406 pad 2: GND -> /UC3843/FB
- R501 pad 1: Net-(NX501-PadA) -> LED
- R501 pad 2: +170V -> /Lamps/TwoDigits1/SK_IN
- R601 pad 1: Net-(NX601-PadA) -> +3V3
- R601 pad 2: +170V -> ~{PWM_DIGITS}
- R701 pad 1: Net-(NX702-PadA) -> +3V3
- R701 pad 2: +170V -> ~{PWM_DIGITS}
- U101 pad 3: /TwoDigits2/Digit2/K155ID1_A -> /Lamps/TwoDigits1/Digit1/K155ID1_A
- U101 pad 4: /TwoDigits2/Digit2/K155ID1_D -> /Lamps/TwoDigits1/Digit1/K155ID1_D
- U101 pad 6: /TwoDigits2/Digit2/K155ID1_B -> /Lamps/TwoDigits1/Digit1/K155ID1_B
- U101 pad 7: /TwoDigits2/Digit2/K155ID1_C -> /Lamps/TwoDigits1/Digit1/K155ID1_C
- U102 pad 3: /TwoDigits3/Digit2/K155ID1_A -> /Lamps/TwoDigits2/Digit1/K155ID1_A
- U102 pad 4: /TwoDigits3/Digit2/K155ID1_D -> /Lamps/TwoDigits2/Digit1/K155ID1_D
- U102 pad 6: /TwoDigits3/Digit2/K155ID1_B -> /Lamps/TwoDigits2/Digit1/K155ID1_B
- U102 pad 7: /TwoDigits3/Digit2/K155ID1_C -> /Lamps/TwoDigits2/Digit1/K155ID1_C
- U104 pad 1: unconnected-(U102-3V3-Pad1) -> +3V3
- U104 pad 15: ~{PWM} -> ~{PWM_DIGITS}
- U104 pad 19: Net-(U102-GND-Pad19) -> GND
- U104 pad 4: unconnected-(U102-GPIO5/ADC2_CH0-Pad4) -> ~{PWM_DOTS}
- U104 pad 7: unconnected-(U102-GPIO8-Pad7) -> DALLAS
- U104 pad 9: Net-(U102-GND-Pad19) -> GND
- U201 pad 3: /TwoDigits3/Digit1/K155ID1_A -> /Lamps/TwoDigits2/Digit2/K155ID1_A
- U201 pad 4: /TwoDigits3/Digit1/K155ID1_D -> /Lamps/TwoDigits2/Digit2/K155ID1_D
- U201 pad 6: /TwoDigits3/Digit1/K155ID1_B -> /Lamps/TwoDigits2/Digit2/K155ID1_B
- U201 pad 7: /TwoDigits3/Digit1/K155ID1_C -> /Lamps/TwoDigits2/Digit2/K155ID1_C
- U202 pad 3: /TwoDigits2/Digit1/K155ID1_A -> /Lamps/TwoDigits1/Digit2/K155ID1_A
- U202 pad 4: /TwoDigits2/Digit1/K155ID1_D -> /Lamps/TwoDigits1/Digit2/K155ID1_D
- U202 pad 6: /TwoDigits2/Digit1/K155ID1_B -> /Lamps/TwoDigits1/Digit2/K155ID1_B
- U202 pad 7: /TwoDigits2/Digit1/K155ID1_C -> /Lamps/TwoDigits1/Digit2/K155ID1_C
- U401 pad 2: Net-(U401-FB) -> /UC3843/FB
- U401 pad 3: Net-(Q401-S) -> Net-(U401-CS)
- U401 pad 7: +12V -> Net-(U401-VCC)
- U601 pad 1: /TwoDigits2/Digit1/K155ID1_B -> /Lamps/TwoDigits1/Digit1/K155ID1_B
- U601 pad 13: ~{PWM} -> ~{PWM_DIGITS}
- U601 pad 14: /TwoDigits1/74HC595_OUT -> MOSI
- U601 pad 15: /TwoDigits2/Digit1/K155ID1_A -> /Lamps/TwoDigits1/Digit1/K155ID1_A
- U601 pad 2: /TwoDigits2/Digit1/K155ID1_C -> /Lamps/TwoDigits1/Digit1/K155ID1_C
- U601 pad 3: /TwoDigits2/Digit1/K155ID1_D -> /Lamps/TwoDigits1/Digit1/K155ID1_D
- U601 pad 4: /TwoDigits2/Digit2/K155ID1_A -> /Lamps/TwoDigits1/Digit2/K155ID1_A
- U601 pad 5: /TwoDigits2/Digit2/K155ID1_B -> /Lamps/TwoDigits1/Digit2/K155ID1_B
- U601 pad 6: /TwoDigits2/Digit2/K155ID1_C -> /Lamps/TwoDigits1/Digit2/K155ID1_C
- U601 pad 7: /TwoDigits2/Digit2/K155ID1_D -> /Lamps/TwoDigits1/Digit2/K155ID1_D
- U701 pad 1: /TwoDigits3/Digit1/K155ID1_B -> /Lamps/TwoDigits2/Digit1/K155ID1_B
- U701 pad 13: ~{PWM} -> ~{PWM_DIGITS}
- U701 pad 15: /TwoDigits3/Digit1/K155ID1_A -> /Lamps/TwoDigits2/Digit1/K155ID1_A
- U701 pad 2: /TwoDigits3/Digit1/K155ID1_C -> /Lamps/TwoDigits2/Digit1/K155ID1_C
- U701 pad 3: /TwoDigits3/Digit1/K155ID1_D -> /Lamps/TwoDigits2/Digit1/K155ID1_D
- U701 pad 4: /TwoDigits3/Digit2/K155ID1_A -> /Lamps/TwoDigits2/Digit2/K155ID1_A
- U701 pad 5: /TwoDigits3/Digit2/K155ID1_B -> /Lamps/TwoDigits2/Digit2/K155ID1_B
- U701 pad 6: /TwoDigits3/Digit2/K155ID1_C -> /Lamps/TwoDigits2/Digit2/K155ID1_C
- U701 pad 7: /TwoDigits3/Digit2/K155ID1_D -> /Lamps/TwoDigits2/Digit2/K155ID1_D
- U701 pad 9: /TwoDigits3/74HC595_OUT -> /Lamps/TwoDigits2/74HC595_OUT
Routing:
- net +170V: track 0.00 -> 39.9 mm
- net Net-(U401-VCC): track 0.00 -> 39.6 mm, vias 0 -> 2
- net /UC3843/PWR_GND: track 0.00 -> 30.2 mm
- net /UC3843/FB: track 0.00 -> 17.9 mm
- net /UC3843/PWR_SW: track 0.00 -> 16.5 mm
- net Net-(NT402-Pad2): track 0.00 -> 14.7 mm, vias 0 -> 2
- net Net-(U401-OUT): track 0.00 -> 14.4 mm
- net Net-(Q401-G): track 0.00 -> 14.0 mm
- net Net-(U401-VREF): track 0.00 -> 11.7 mm
- net +12V: track 0.00 -> 11.2 mm
- net /UC3843/PWR_SEN: track 0.00 -> 9.72 mm
- net Net-(U401-RC): track 0.00 -> 8.48 mm
- net Net-(U401-COMP): track 0.00 -> 7.05 mm
- net (no net): vias 2 -> 0
- added copper zone on B.Cu, net /UC3843/PWR_GND
- added copper zone on F.Cu, net /UC3843/PWR_GND
Other:
- board size 309 x 88 mm -> 146.2 x 85.8 mm
- board text removed: "Top"
