File: hardware/NosClock.kicad_pcb (KiCad board)
At the start: 2 copper layers, 146.2 x 85.8 mm, 129 parts, among them J101 AC, J102 USB_C_Receptacle_USB2.0_16P, Q401 AOD11S60, Q901 MMBTA42, Q902 MMBTA42, Q903 MMBTA42, Q904 MMBTA42, U101 K155ID1, U102 K155ID1, U103 DS18B20, U104 ESP32-C3-WROOM-02, U201 K155ID1, U202 K155ID1, U203 MP2307DN-LF-Z, U301 AP7361-33ER-13, U401 UC3843_SOIC8, U601 74HC595, U701 74HC595, U801 74HC595, U802 K155ID1, U803 K155ID1, U901 74HC595

Commit message: 2/static version
Parts:
- removed C102, C103, C104, C105, C211, C801, C802, C803, C804: 100nF, Capacitor_SMD:C_0603_1608Metric
- removed the C207 at (92.5, 100.0)
- removed the C208 at (42.5, 99.5)
- removed the C210 at (56.6, 99.5)
- removed the C301 at (-17.9, 160.4)
- removed the C302 at (-22.5, 160.6)
- removed the C303 at (-17.9, 162.9)
- removed D101, D102, D103, D104, D201, D202, D203, D204, D801, D802, D803, D804: SK6812MINI_ALI, LED_SMD:LED_SK6812MINI_PLCC4_3.5x3.5mm_P1.75mm
- removed the J101 at (43.5, 140.7)
- removed N901, N902, N903, N904: INS-1, mynixies:mynixies-INS-1
- removed NX101, NX102, NX201, NX202, NX801, NX802: IN-12B, nixies-us:nixies-us-IN-12
- removed Q903, Q904: MMBTA42, Package_TO_SOT_SMD:SOT-23
- removed the R101 at (59.5, 219.9)
- removed the R106 at (122.6, 126.4)
- removed R107: 22K, Resistor_SMD:R_2512_6332Metric
- removed the R202 at (46.6, 125.9)
- removed the R203 at (96.6, 126.4)
- removed R905: 10K, Resistor_SMD:R_0603_1608Metric
- removed R906, R907, R908, R909: 47K, Resistor_SMD:R_0603_1608Metric
- removed R910, R911, R912, R913: 330K, Resistor_SMD:R_1206_3216Metric
- removed the TP_101 at (63.2, 220.2)
- removed the U102 at (129.3, 87.0)
- removed U104: ESP32-C3-WROOM-02, PCM_Espressif:ESP32-C3-WROOM-02
- removed the U202 at (57.6, 86.5)
- removed the U301 at (-20.0, 155.0)
- removed U701, U801, U901: 74HC595, Package_SO:TSSOP-16_4.4x5mm_P0.65mm
- removed U802, U803: K155ID1, Package_DIP:DIP-16_W7.62mm
- added C202: 100nF, Capacitor_SMD:C_0603_1608Metric, F.Cu at (105.2, 98.2)
- added C203: 100nF, Capacitor_SMD:C_0603_1608Metric, F.Cu at (103.2, 114.2)
- added C204: 10uF, Capacitor_SMD:C_0805_2012Metric, F.Cu at (99.6, 114.0)
- added C401: 100uF 10V, Capacitor_THT:CP_Radial_D6.3mm_P2.50mm, F.Cu at (72.3, 58.9)
- added C502: 100nF, Capacitor_SMD:C_0603_1608Metric, F.Cu at (78.2, 90.4)
- added C503: 100nF, Capacitor_SMD:C_0603_1608Metric, F.Cu at (99.6, 70.2)
- added C504: 100nF, Capacitor_SMD:C_0603_1608Metric, F.Cu at (98.3, 90.4)
- added C505: 100nF, Capacitor_SMD:C_0603_1608Metric, F.Cu at (129.5, 70.2)
- added C506: 100nF, Capacitor_SMD:C_0603_1608Metric, F.Cu at (128.2, 90.4)
- added C601: 100nF, Capacitor_SMD:C_0603_1608Metric, F.Cu at (149.6, 70.2)
- added C602: 100nF, Capacitor_SMD:C_0603_1608Metric, F.Cu at (148.3, 90.4)
- added C603: 100nF, Capacitor_SMD:C_0603_1608Metric, F.Cu at (179.6, 70.2)
- added C604: 100nF, Capacitor_SMD:C_0603_1608Metric, F.Cu at (178.2, 90.4)
- added C605: 100nF, Capacitor_SMD:C_0603_1608Metric, F.Cu at (197.9, 69.1)
- added C606: 100nF, Capacitor_SMD:C_0603_1608Metric, F.Cu at (197.4, 90.4)
- added D401: ES1J, Diode_SMD:D_SMA, F.Cu at (80.7, 59.1)
- added D502: SK6812MINI_ALI, LED_SMD:LED_SK6812MINI_PLCC4_3.5x3.5mm_P1.75mm, F.Cu at (70.3, 84.2)
- added D503: SK6812MINI_ALI, LED_SMD:LED_SK6812MINI_PLCC4_3.5x3.5mm_P1.75mm, F.Cu at (90.4, 74.6)
- added D504: SK6812MINI_ALI, LED_SMD:LED_SK6812MINI_PLCC4_3.5x3.5mm_P1.75mm, F.Cu at (90.4, 84.2)
- added D505: SK6812MINI_ALI, LED_SMD:LED_SK6812MINI_PLCC4_3.5x3.5mm_P1.75mm, F.Cu at (120.3, 74.6)
- added D506: SK6812MINI_ALI, LED_SMD:LED_SK6812MINI_PLCC4_3.5x3.5mm_P1.75mm, F.Cu at (120.3, 84.2)
- added D601: SK6812MINI_ALI, LED_SMD:LED_SK6812MINI_PLCC4_3.5x3.5mm_P1.75mm, F.Cu at (140.4, 74.6)
- added D602: SK6812MINI_ALI, LED_SMD:LED_SK6812MINI_PLCC4_3.5x3.5mm_P1.75mm, F.Cu at (140.4, 84.2)
- added D603: SK6812MINI_ALI, LED_SMD:LED_SK6812MINI_PLCC4_3.5x3.5mm_P1.75mm, F.Cu at (170.3, 74.6)
- added D604: SK6812MINI_ALI, LED_SMD:LED_SK6812MINI_PLCC4_3.5x3.5mm_P1.75mm, F.Cu at (170.3, 84.2)
- added D605: SK6812MINI_ALI, LED_SMD:LED_SK6812MINI_PLCC4_3.5x3.5mm_P1.75mm, F.Cu at (190.4, 74.6)
- added D606: SK6812MINI_ALI, LED_SMD:LED_SK6812MINI_PLCC4_3.5x3.5mm_P1.75mm, F.Cu at (190.4, 84.2)
- added H101: MountingHole, MountingHole:MountingHole_3.2mm_M3_Pad_Via, F.Cu at (63.0, 56.5)
- added H102: MountingHole, MountingHole:MountingHole_3.2mm_M3_Pad_Via, F.Cu at (63.0, 112.5)
- added H103: MountingHole, MountingHole:MountingHole_3.2mm_M3_Pad_Via, F.Cu at (197.0, 56.5)
- added H104: MountingHole, MountingHole:MountingHole_3.2mm_M3_Pad_Via, F.Cu at (197.0, 112.4)
- added J102: 12V IN, Connector_JST:JST_XH_B2B-XH-A_1x02_P2.50mm_Vertical, F.Cu at (131.6, 113.5)
- added N401: INS-1, mynixies:mynixies-INS-1, F.Cu at (105.2, 74.5)
- added N402: INS-1, mynixies:mynixies-INS-1, F.Cu at (105.2, 84.3)
- added N403: INS-1, mynixies:mynixies-INS-1, F.Cu at (155.2, 74.5)
- added N404: INS-1, mynixies:mynixies-INS-1, F.Cu at (155.2, 84.8)
- added NT102: NetTie_2, NetTie:NetTie-2_SMD_Pad0.5mm, F.Cu at (154.8, 100.0)
- added NT103: NetTie_2, NetTie:NetTie-2_SMD_Pad0.5mm, F.Cu at (98.4, 113.1)
- added NT104: NetTie_2, NetTie:NetTie-2_SMD_Pad0.5mm, F.Cu at (109.4, 97.0)
- added NX501: IN-12B, nixies-us:nixies-us-IN-12, F.Cu at (70.6, 79.4)
- added NX502: IN-12B, nixies-us:nixies-us-IN-12, F.Cu at (90.8, 79.4)
- added NX503: IN-12B, nixies-us:nixies-us-IN-12, F.Cu at (120.6, 79.4)
- added NX601: IN-12B, nixies-us:nixies-us-IN-12, F.Cu at (140.8, 79.4)
- added NX602: IN-12B, nixies-us:nixies-us-IN-12, F.Cu at (170.6, 79.4)
- added NX603: IN-12B, nixies-us:nixies-us-IN-12, F.Cu at (190.8, 79.4)
- added Q401: MPSA42, Package_TO_SOT_THT:TO-92_Inline, F.Cu at (130.9, 95.9)
- added Q701: MPSA92, Package_TO_SOT_THT:TO-92_Inline, F.Cu at (196.2, 99.0)
- added Q702: MPSA42, Package_TO_SOT_THT:TO-92_Inline, F.Cu at (182.9, 114.3)
- added Q801: MPSA92, Package_TO_SOT_THT:TO-92_Inline, F.Cu at (196.2, 93.4)
- added Q802: MPSA42, Package_TO_SOT_THT:TO-92_Inline, F.Cu at (182.8, 99.6)
- added R102: 4.7K, Resistor_SMD:R_0603_1608Metric_Pad0.98x0.95mm_HandSolder, F.Cu at (97.1, 98.2)
- added R103: 4.7K, Resistor_SMD:R_0603_1608Metric_Pad0.98x0.95mm_HandSolder, F.Cu at (97.1, 94.6)
- added R401: 330K, Resistor_SMD:R_1206_3216Metric, F.Cu at (105.2, 68.5)
- added R402: 330K, Resistor_SMD:R_1206_3216Metric, F.Cu at (105.2, 92.1)
- added R403: 10K, Resistor_SMD:R_0603_1608Metric, F.Cu at (131.3, 103.0)
- added R404: 47K, Resistor_SMD:R_0603_1608Metric, F.Cu at (134.6, 103.0)
- added R405: 330K, Resistor_SMD:R_1206_3216Metric, F.Cu at (155.2, 68.5)
- added R406: 330R, Resistor_SMD:R_0603_1608Metric, F.Cu at (68.4, 95.2)
- added R407: 330K, Resistor_SMD:R_1206_3216Metric, F.Cu at (155.6, 92.1)
- added R502: 22K, Resistor_SMD:R_2512_6332Metric, F.Cu at (176.8, 58.4)
- added R503: 22K, Resistor_SMD:R_2512_6332Metric, F.Cu at (186.8, 58.4)
- added R602: 22K, Resistor_SMD:R_2512_6332Metric, F.Cu at (176.8, 64.1)
- added R603: 22K, Resistor_SMD:R_2512_6332Metric, F.Cu at (186.8, 64.1)
- added R702: 220K, Resistor_SMD:R_1206_3216Metric, F.Cu at (187.6, 113.0)
- added R703: 10K, Resistor_SMD:R_0603_1608Metric, F.Cu at (176.7, 111.0)
- added R704: 47K, Resistor_SMD:R_0603_1608Metric, F.Cu at (176.7, 115.0)
- added R804: 47K, Resistor_SMD:R_0603_1608Metric, F.Cu at (176.7, 100.3)
- added TP_102: SDA, NosLib:TestPoint_Pad_1.0x1.0mm, F.Cu at (93.6, 94.6)
- added TP_104: SCL, NosLib:TestPoint_Pad_1.0x1.0mm, F.Cu at (93.6, 98.2)
- added U401: 74HC595, Package_SO:TSSOP-16_4.4x5mm_P0.65mm, F.Cu at (127.4, 60.5)
- added U501: K155ID1, Package_DIP:DIP-16_W7.62mm, F.Cu at (104.2, 64.1)
- C303: renamed from C405; value 4.7uF 250V -> 4.7uF 400V
- C501: value 100uF 10V -> 100nF; footprint Capacitor_THT:CP_Radial_D6.3mm_P2.50mm -> Capacitor_SMD:C_0603_1608Metric
- D501: value ES1J -> SK6812MINI_ALI; footprint Diode_SMD:D_SMA_Handsoldering -> LED_SMD:LED_SK6812MINI_PLCC4_3.5x3.5mm_P1.75mm
- NT101: moved to B.Cu
- Q901: value MMBTA42 -> MPSA92; footprint Package_TO_SOT_SMD:SOT-23 -> Package_TO_SOT_THT:TO-92_Inline
- Q902: value MMBTA42 -> MPSA42; footprint Package_TO_SOT_SMD:SOT-23 -> Package_TO_SOT_THT:TO-92_Inline
- R501: value 330R -> 22K; footprint Resistor_SMD:R_0603_1608Metric -> Resistor_SMD:R_2512_6332Metric
- R601: value 10K -> 22K; footprint Resistor_SMD:R_0603_1608Metric -> Resistor_SMD:R_2512_6332Metric
- R701, R801, R901, R902: value 10K -> 220K; footprint Resistor_SMD:R_0603_1608Metric -> Resistor_SMD:R_1206_3216Metric
- R802: value 22K -> 220K; footprint Resistor_SMD:R_2512_6332Metric -> Resistor_SMD:R_1206_3216Metric
- R803: value 22K -> 10K; footprint Resistor_SMD:R_2512_6332Metric -> Resistor_SMD:R_0603_1608Metric
- R904: value 10K -> 47K
- U101: value K155ID1 -> ESP32-C3-WROOM-02; footprint Package_DIP:DIP-16_W7.62mm -> PCM_Espressif:ESP32-C3-WROOM-02
- U201: value K155ID1 -> AP7361-33ER-13; footprint Package_DIP:DIP-16_W7.62mm -> Package_TO_SOT_SMD:SOT-223-3_TabPin2
- U601: value 74HC595 -> K155ID1; footprint Package_SO:TSSOP-16_4.4x5mm_P0.65mm -> Package_DIP:DIP-16_W7.62mm
- moved R901 201.3 mm to (191.5, 105.8), turned to -90 degrees
- moved C201 156.8 mm to (126.5, 101.0), turned to 90 degrees
- moved R201 156.5 mm to (126.5, 106.0), turned to -90 degrees
- moved C209 155.4 mm to (126.5, 111.0), turned to 90 degrees
- moved R204 155.0 mm to (125.8, 115.0), turned to 180 degrees
- moved C205 146.9 mm to (120.9, 98.2), turned to 180 degrees
- moved C206 146.7 mm to (120.9, 102.1), turned to 180 degrees
- moved R203 146.4 mm to (116.8, 115.0), turned to 180 degrees
- moved C210 145.9 mm to (121.3, 115.0)
- moved R202 142.3 mm to (112.4, 115.0), turned to 180 degrees
- moved NT202 141.2 mm to (125.6, 100.2), turned to 180 degrees
- moved U202 140.7 mm to (121.4, 108.8), turned to -90 degrees
- moved C208 140.7 mm to (112.0, 98.2)
- moved NT201 140.4 mm to (126.3, 104.3), turned to -90 degrees
- moved C207 139.1 mm to (112.0, 102.1)
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- renumbered C205 to C201, C201 to C205, C202 to C206, C206 to C207, C209 to C208, C203 to C209, C204 to C210, C401 to C301, C402 to C302, C406 to C304, C404 to C305, C403 to C306, D401 to D301, J102 to J101, L401 to L301, NT102 to NT105, NT203 to NT202, NT204 to NT203, NT202 to NT204, NT401 to NT301, NT403 to NT302, NT402 to NT303, Q401 to Q301, R102 to R101, R103 to R104, R104 to R105, R105 to R106, R206 to R202, R205 to R203, R401 to R301, R404 to R302, R406 to R303, R403 to R304, R402 to R305, R405 to R306, R407 to R307, TP_102 to TP_101, U103 to U102, U203 to U202, U401 to U301
Connections:
- net +12V renamed /MP2307/+12V
- C207 pad 1: +5V -> /MP2307/+5V
- C208 pad 1: +5V -> /MP2307/+5V
- C303 pad 1: +170V -> /UC3843/+170V
- C501 pad 1: GND -> /Lamps/FIRST_SK6812MINI_VCC
- C501 pad 2: +5V -> GND
- D301 pad 1: +170V -> /UC3843/+170V
- D501 pad 1: /Lamps/TwoDigits1/FIRST_SK6812MINI_VCC -> /Lamps/FIRST_SK6812MINI_VCC
- D501 pad 2: +5V -> Net-(D501-DOUT)
- L201 pad 2: +5V -> /MP2307/+5V
- NT101 pad 2: 5V -> +5V
- NT203 pad 2: +5V -> /MP2307/+5V
- NT302 pad 1: +170V -> /UC3843/+170V
- Q901 pad 1: Net-(Q901-B) -> +170V
- Q901 pad 2: GND -> Net-(Q901-B)
- Q901 pad 3: Net-(Q901-C) -> /Lamps/HighSideSwitch3/VOUT
- Q902 pad 1: Net-(Q902-B) -> GND
- Q902 pad 2: GND -> Net-(Q902-B)
- R101 pad 1: 3V3 -> +3V3
- R501 pad 1: LED -> Net-(NX501-PadA)
- R501 pad 2: /Lamps/TwoDigits1/SK_IN -> /Lamps/HighSideSwitch3/VOUT
- R601 pad 1: +3V3 -> Net-(NX601-PadA)
- R601 pad 2: ~{PWM_DIGITS} -> /Lamps/HighSideSwitch3/VOUT
- R701 pad 1: +3V3 -> +170V
- R701 pad 2: ~{PWM_DIGITS} -> Net-(Q701-B)
- R801 pad 1: +3V3 -> +170V
- R801 pad 2: ~{PWM_DIGITS} -> Net-(Q801-B)
- R802 pad 2: +170V -> Net-(Q801-B)
- R803 pad 1: Net-(NX802-PadA) -> MUX2
- R803 pad 2: +170V -> Net-(Q802-B)
- R901 pad 1: +3V3 -> +170V
- R901 pad 2: ~{PWM_DOTS} -> Net-(Q901-B)
- R902 pad 1: /Lamps/Dots/Dot3/EN -> Net-(Q902-C)
- R902 pad 2: Net-(Q902-B) -> Net-(Q901-B)
- R903 pad 1: /Lamps/Dots/Dot1/EN -> MUX3
- R903 pad 2: Net-(Q901-B) -> Net-(Q902-B)
- R904 pad 1: /Lamps/Dots/Dot2/EN -> GND
- R904 pad 2: Net-(Q904-B) -> Net-(Q902-B)
- U101 pad 1: Net-(U101-~{Q8}) -> +3V3
- U101 pad 10: Net-(U101-~{Q7}) -> CS
- U101 pad 11: Net-(U101-~{Q6}) -> INPUT
- U101 pad 12: GND -> SK6812MINI_DATA
- U101 pad 13: Net-(U101-~{Q4}) -> USB_D-
- U101 pad 14: Net-(U101-~{Q5}) -> USB_D+
- U101 pad 15: Net-(U101-~{Q1}) -> MUX3
- U101 pad 16: Net-(U101-~{Q0}) -> DALLAS
- U101 pad 2: Net-(U101-~{Q9}) -> EN
- U101 pad 3: /Lamps/TwoDigits1/Digit1/K155ID1_A -> INPUT2
- U101 pad 4: /Lamps/TwoDigits1/Digit1/K155ID1_D -> COLONS
- U101 pad 5: +5V -> SCK
- U101 pad 6: /Lamps/TwoDigits1/Digit1/K155ID1_B -> MOSI
- U101 pad 7: /Lamps/TwoDigits1/Digit1/K155ID1_C -> SDA
- U101 pad 8: Net-(U101-~{Q2}) -> SCL
- U101 pad 9: Net-(U101-~{Q3}) -> GND
- U201 pad 1: Net-(U201-~{Q8}) -> GND
- U201 pad 2: Net-(U201-~{Q9}) -> /MP2307/+3V3
- U201 pad 3: /Lamps/TwoDigits2/Digit2/K155ID1_A -> /MP2307/+5V
- U202 pad 4: GND -> /MP2307/PWR_GND
- U601 pad 1: /Lamps/TwoDigits1/Digit1/K155ID1_B -> /Lamps/ThreeDigits2/NX8
- U601 pad 10: +3V3 -> /Lamps/ThreeDigits2/NX7
- U601 pad 11: SCK -> /Lamps/ThreeDigits2/NX6
- U601 pad 12: CS -> GND
- U601 pad 13: ~{PWM_DIGITS} -> /Lamps/ThreeDigits2/NX4
- U601 pad 14: MOSI -> /Lamps/ThreeDigits2/NX5
- U601 pad 15: /Lamps/TwoDigits1/Digit1/K155ID1_A -> /Lamps/ThreeDigits2/NX1
- U601 pad 16: +3V3 -> /Lamps/ThreeDigits2/NX0
- U601 pad 2: /Lamps/TwoDigits1/Digit1/K155ID1_C -> /Lamps/ThreeDigits2/NX9
- U601 pad 3: /Lamps/TwoDigits1/Digit1/K155ID1_D -> /Lamps/ThreeDigits2/DIGIT_A
- U601 pad 4: /Lamps/TwoDigits1/Digit2/K155ID1_A -> /Lamps/ThreeDigits2/DIGIT_D
- U601 pad 5: /Lamps/TwoDigits1/Digit2/K155ID1_B -> +5V
- U601 pad 6: /Lamps/TwoDigits1/Digit2/K155ID1_C -> /Lamps/ThreeDigits2/DIGIT_B
- U601 pad 7: /Lamps/TwoDigits1/Digit2/K155ID1_D -> /Lamps/ThreeDigits2/DIGIT_C
- U601 pad 8: GND -> /Lamps/ThreeDigits2/NX2
- U601 pad 9: /Lamps/TwoDigits1/74HC595_OUT -> /Lamps/ThreeDigits2/NX3
Routing:
- net +5V: track 0.00 -> 436.2 mm, vias 0 -> 21
- net GND: track 0.00 -> 173.4 mm, vias 0 -> 23
- net /Lamps/ThreeDigits2/NX1: track 0.00 -> 144.8 mm, vias 0 -> 2
- net /Lamps/ThreeDigits2/NX0: track 0.00 -> 143.1 mm, vias 0 -> 2
- net MUX1: track 0.00 -> 140.5 mm, vias 0 -> 2
- net /Lamps/ThreeDigits1/NX2: track 0.00 -> 132.7 mm, vias 0 -> 3
- net /Lamps/ThreeDigits1/NX1: track 0.00 -> 130.6 mm, vias 0 -> 2
- net /Lamps/ThreeDigits2/NX9: track 0.00 -> 126.3 mm, vias 0 -> 2
- net +170V: track 39.9 -> 165.9 mm, vias 0 -> 3
- net /Lamps/ThreeDigits2/NX3: track 0.00 -> 124.4 mm, vias 0 -> 2
- net MUX2: track 0.00 -> 123.3 mm, vias 0 -> 2
- net /Lamps/ThreeDigits1/NX3: track 0.00 -> 121.5 mm, vias 0 -> 2
- net MUX3: track 0.00 -> 120.4 mm, vias 0 -> 4
- net /Lamps/ThreeDigits2/NX8: track 0.00 -> 119.6 mm, vias 0 -> 2
- net Net-(NX501-PadA): track 0.00 -> 118.9 mm, vias 0 -> 3
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- added copper zone on B.Cu, net /MP2307/PWR_GND
- added copper zone on F.Cu, net /MP2307/PWR_GND
- added copper zone on B.Cu, net GND
- added copper zone on F.Cu, net GND
- removed copper zone on B.Cu, net /UC3843/PWR_GND
- removed copper zone on F.Cu, net /UC3843/PWR_GND
Other:
- board size 146.2 x 85.8 mm -> 142 x 64 mm

Commit message: Battery
Parts:
- removed the TP_103 at (68.9, 113.4)
- added BT101: Battery_Cell, NosLib:BAT_CH291-1220LF, F.Cu at (82.5, 60.4)
- added C102: 100nF, Capacitor_SMD:C_0603_1608Metric, F.Cu at (97.5, 54.9)
- added J102: Conn_01x04, Connector_Molex:Molex_PicoBlade_53047-0410_1x04_P1.25mm_Vertical, F.Cu at (73.5, 54.8)
- added TP_102: GND, NosLib:TestPoint_Pad_1.0x1.0mm, F.Cu at (96.4, 109.7)
- added TP_105: +170V, NosLib:TestPoint_Pad_1.0x1.0mm, F.Cu at (93.0, 131.9)
- added TP_106: +5V, NosLib:TestPoint_Pad_1.0x1.0mm, F.Cu at (95.1, 137.2)
- added TP_107: +3V3, NosLib:TestPoint_Pad_1.0x1.0mm, F.Cu at (98.2, 134.1)
- added TP_108: +12V, NosLib:TestPoint_Pad_1.0x1.0mm, F.Cu at (98.2, 137.2)
- added U103: DS3231MZ, Package_SO:SOIC-8_3.9x4.9mm_P1.27mm, F.Cu at (97.5, 61.0)
- moved D401 19.7 mm to (61.8, 64.3), turned to -90 degrees
- moved C401 4.41 mm to (68.8, 61.6), turned to 180 degrees
- moved TP_101 0.84 mm to (96.3, 112.9), turned to 0 degrees
- moved H103 0.65 mm to (197.0, 55.8)
- moved H101 0.63 mm to (63.0, 55.8)
- renumbered J102 to J103, TP_102 to TP_103
Connections:
- net /MP2307/+12V renamed +12V
Routing:
- net SCL: track 7.65 -> 90.3 mm, vias 0 -> 4
- net SDA: track 6.48 -> 88.5 mm
- net +3V3: track 110.5 -> 189.0 mm, vias 4 -> 7
- net /Lamps/FIRST_SK6812MINI_VCC: track 21.3 -> 36.4 mm, vias 2 -> 5
- net GND: track 173.4 -> 182.8 mm, vias 23 -> 25
- net Net-(BT101-+): track 0.00 -> 7.80 mm
- net +5V: track 436.2 -> 432.1 mm, vias 21 -> 19
- net /Lamps/ThreeDigits1/NX4: track 98.5 -> 96.2 mm
- net /Lamps/ThreeDigits1/NX5: track 85.8 -> 84.7 mm
- net Net-(NX501-PadA): track 118.9 -> 117.8 mm
- net /Lamps/ThreeDigits1/DIGIT_C: track 15.7 -> 16.4 mm
- net Net-(NX503-PadA): track 91.5 -> 90.9 mm
Other:
- board size 142 x 64 mm -> 142 x 64.6 mm

Commit message: Finalize schematics
Parts:
- removed the NT102 at (154.8, 100.0)
- removed the NT202 at (125.6, 100.2)
- added C101: 100nF, Capacitor_SMD:C_0603_1608Metric, F.Cu at (101.7, 107.1)
- added J103: Conn_01x02, Connector_JST:JST_PH_B2B-PH-K_1x02_P2.00mm_Vertical, F.Cu at (71.7, 112.4)
- added TP_101: DBG, NosLib:TestPoint_Pad_1.0x1.0mm, F.Cu at (107.4, 111.0)
- added TP_102: GND, NosLib:TestPoint_Pad_1.0x1.0mm, F.Cu at (113.7, 114.7)
- added TP_111: GND, NosLib:TestPoint_Pad_1.0x1.0mm, F.Cu at (172.5, 91.8)
- C303: footprint Capacitor_THT:CP_Radial_D8.0mm_P3.50mm -> Capacitor_THT:CP_Radial_D10.0mm_P5.00mm
- N401, N402, N403, N404: footprint mynixies:mynixies-INS-1 -> NosLib:INS-1
- NT101: moved to F.Cu
- NX501, NX502, NX503, NX601, NX602, NX603: footprint nixies-us:nixies-us-IN-12 -> NosLib:nixies-us-IN-12
- Q701, Q801, Q901: value MPSA92 -> MMBTA92; footprint Package_TO_SOT_THT:TO-92_Inline -> Package_TO_SOT_SMD:SOT-23
- Q702, Q802, Q902: value MPSA42 -> MMBTA42; footprint Package_TO_SOT_THT:TO-92_Inline -> Package_TO_SOT_SMD:SOT-23
- R501, R502, R503, R601, R602, R603: value 22K -> 4.7K; footprint Resistor_SMD:R_2512_6332Metric -> Resistor_SMD:R_1206_3216Metric
- TP_107: renamed from TP_105; value +170V -> 170V
- TP_108: renamed from TP_106; value +5V -> 5V
- TP_109: renamed from TP_107; value +3V3 -> 3V3
- TP_110: renamed from TP_108; value +12V -> 12V
- moved TP_107 83.4 mm to (166.0, 91.8)
- moved TP_110 80.2 mm to (166.0, 94.3)
- moved TP_108 79.3 mm to (160.2, 91.8)
- moved J101 75.7 mm to (121.8, 113.1)
- moved TP_109 73.7 mm to (160.2, 94.3)
- moved R901 65.3 mm to (144.6, 60.5), turned to 0 degrees
- moved Q901 65.1 mm to (144.6, 65.0), turned to 180 degrees
- moved BT101 59.3 mm to (127.8, 98.8), turned to 0 degrees
- moved R902 59.2 mm to (149.6, 60.5), turned to 180 degrees
- moved R704 56.7 mm to (192.2, 60.5), turned to -90 degrees
- moved Q902 53.7 mm to (149.6, 65.0), turned to 180 degrees
- moved R701 53.4 mm to (182.5, 60.5), turned to 0 degrees
- moved C103 52.9 mm to (107.0, 106.9), turned to 0 degrees
- moved R702 52.6 mm to (187.4, 60.5), turned to 180 degrees
- moved R904 52.4 mm to (154.3, 60.5), turned to -90 degrees
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- renumbered C101 to C102, C102 to C103, J102 to J101, J101 to J102, J103 to J104, NT103 to NT102, NT104 to NT103, NT105 to NT104, NT203 to NT202, NT204 to NT203, TP_101 to TP_103, TP_102 to TP_104, TP_103 to TP_105, TP_104 to TP_106
Connections:
- net /Lamps/FIRST_SK6812MINI_VCC renamed /Lamps/ThreeDigits1/FIRST_SK6812MINI_VCC
- C201 pad 2: Net-(C201-Pad2) -> /MP2307/SW
- C303 pad 1: /UC3843/+170V -> +170V
- D301 pad 1: /UC3843/+170V -> +170V
- NT302 pad 1: /UC3843/+170V -> +170V
- Q701 pad 1: +170V -> Net-(Q701-B)
- Q701 pad 2: Net-(Q701-B) -> +170V
- Q702 pad 1: GND -> Net-(Q702-B)
- Q702 pad 2: Net-(Q702-B) -> GND
- Q801 pad 1: +170V -> Net-(Q801-B)
- Q801 pad 2: Net-(Q801-B) -> +170V
- Q802 pad 1: GND -> Net-(Q802-B)
- Q802 pad 2: Net-(Q802-B) -> GND
- Q901 pad 1: +170V -> Net-(Q901-B)
- Q901 pad 2: Net-(Q901-B) -> +170V
- Q902 pad 1: GND -> Net-(Q902-B)
- Q902 pad 2: Net-(Q902-B) -> GND
- U101 pad 3: INPUT2 -> DBG
Routing:
- net /Lamps/HighSideSwitch3/VOUT: track 82.4 -> 7.16 mm, vias 2 -> 0
- net /Lamps/HighSideSwitch2/VOUT: track 58.8 -> 7.11 mm, vias 2 -> 0
- net /Lamps/HighSideSwitch1/VOUT: track 54.2 -> 7.22 mm, vias 2 -> 0
- net /Lamps/ThreeDigits2/NX3: track 124.4 -> 78.2 mm, vias 2 -> 0
- net COLONS: track 48.3 -> 3.69 mm, vias 2 -> 0
- net /Lamps/ThreeDigits2/NX2: track 117.6 -> 74.1 mm, vias 4 -> 1
- net CS: track 92.8 -> 50.6 mm
- net /Lamps/ThreeDigits2/NX1: track 144.8 -> 104.3 mm, vias 2 -> 1
- net DALLAS: track 56.2 -> 17.1 mm, vias 2 -> 1
- net +5V: track 432.1 -> 394.6 mm, vias 19 -> 18
- net SCL: track 90.3 -> 54.8 mm
- net Net-(Q701-B): track 41.1 -> 8.25 mm, vias 1 -> 0
- net SDA: track 88.5 -> 55.6 mm, vias 0 -> 3
- net MOSI: track 76.6 -> 43.8 mm, vias 2 -> 0
- net /Lamps/ThreeDigits2/NX0: track 143.1 -> 110.6 mm, vias 2 -> 3
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Other:
- board size 142 x 64.6 mm -> 142 x 61.5 mm
- board text added: "3V3"
- board text added: "GND"
- board text added: "IN12V"
- board text added: "IO20"
- board text added: "SCL"
- board text added: "SDA"

Commit message: Add logo
Parts:
- added G***: LOGO, LOGO, F.Cu at (71.5, 61.8)
Other:
- board text added: "v1.0"
