File: hardware/NosClock.kicad_pcb (KiCad board)
At the start: 2 copper layers, 142 x 61.5 mm, 148 parts, among them J101 Conn_01x04, J102 USB_C_Receptacle_USB2.0_16P, J103 Conn_01x02, J104 12V IN, Q301 AOD11S60, Q401 MPSA42, Q701 MMBTA92, Q702 MMBTA42, Q801 MMBTA92, Q802 MMBTA42, Q901 MMBTA92, Q902 MMBTA42, U101 ESP32-C3-WROOM-02, U102 DS18B20, U103 DS3231MZ, U201 AP7361-33ER-13, U202 MP2307DN-LF-Z, U301 UC3843_SOIC8, U401 74HC595, U501 K155ID1, U601 K155ID1

Commit message: Fixes
Parts:
- removed Q401: MPSA42, Package_TO_SOT_THT:TO-92_Inline
- added Q402: MMBTA42, Package_TO_SOT_SMD:SOT-23, F.Cu at (114.0, 98.0)
- added R308: 0.25R, Resistor_SMD:R_2512_6332Metric, F.Cu at (168.2, 99.8)
- L301: footprint Inductor_SMD:L_APV_APH1030 -> Inductor_SMD:L_Chilisin_BMRF00101040
- Q301: value AOD11S60 -> FQD12N20L
- R102, R103: footprint Resistor_SMD:R_0603_1608Metric_Pad0.98x0.95mm_HandSolder -> Resistor_SMD:R_0603_1608Metric
- R306: value 0.5R -> 0.25R
- moved NT201 5.08 mm to (163.3, 108.8), turned to 180 degrees
- moved C304 4.58 mm to (162.5, 101.0)
- moved NT104 4.58 mm to (161.4, 98.5)
- moved C201 4.51 mm to (162.1, 105.8), turned to 0 degrees
- moved R201 2.78 mm to (162.1, 108.8), turned to 180 degrees
- moved C209 0.75 mm to (162.1, 111.7), turned to 0 degrees
- moved R306 0.70 mm to (173.1, 99.7)
Connections:
- R306 pad 2: /UC3843/PWR_GND -> Net-(R306-Pad2)
Routing:
- net /UC3843/PWR_GND: track 57.4 -> 27.7 mm
- net +12V: track 60.8 -> 38.4 mm
- net Net-(U202-EN): track 11.9 -> 0.00 mm
- net /UC3843/PWR_SEN: track 12.0 -> 2.28 mm
- net GND: track 172.2 -> 162.5 mm, vias 20 -> 18
- net Net-(U202-BS): track 6.09 -> 0.00 mm, vias 2 -> 0
- net /MP2307/SW: track 14.9 -> 8.87 mm, vias 3 -> 2
- net Net-(U202-SS): track 3.41 -> 0.33 mm
- net Net-(Q402-B): track 15.9 -> 13.7 mm
- net Net-(NT201-Pad2): track 0.84 -> 0.00 mm

Commit message: Lamps tracing
Parts:
- removed D401: ES1J, Diode_SMD:D_SMA
- removed N401, N402, N403, N404: INS-1, NosLib:INS-1
- removed Q402, Q702, Q802, Q902: MMBTA42, Package_TO_SOT_SMD:SOT-23
- removed Q701, Q801, Q901: MMBTA92, Package_TO_SOT_SMD:SOT-23
- removed R402, R405, R407: 330K, Resistor_SMD:R_1206_3216Metric
- removed R403, R703, R803, R903: 10K, Resistor_SMD:R_0603_1608Metric
- removed R404, R704, R804, R904: 47K, Resistor_SMD:R_0603_1608Metric
- removed R406: 330R, Resistor_SMD:R_0603_1608Metric
- removed R702, R801, R802, R901, R902: 220K, Resistor_SMD:R_1206_3216Metric
- removed the TP_101 at (107.4, 111.0)
- removed the TP_102 at (113.7, 114.7)
- added C402: 100nF, Capacitor_SMD:C_0603_1608Metric, F.Cu at (-23.3, 58.3)
- added C501: 100nF, Capacitor_SMD:C_0603_1608Metric, F.Cu at (-23.3, 74.3)
- added C601: 100nF, Capacitor_SMD:C_0603_1608Metric, F.Cu at (-23.3, 69.8)
- added C701: 100nF, Capacitor_SMD:C_0603_1608Metric, F.Cu at (94.7, 33.0)
- added C702: 10uF, Capacitor_SMD:C_0805_2012Metric, F.Cu at (94.9, 38.3)
- added D701: LED_RAGB, LED_THT:LED_D5.0mm-4_RGB, F.Cu at (103.8, 74.9)
- added D702: LED_RAGB, LED_THT:LED_D5.0mm-4_RGB, F.Cu at (103.8, 83.9)
- added D703: LED_RAGB, LED_THT:LED_D5.0mm-4_RGB, F.Cu at (153.8, 74.9)
- added D704: LED_RAGB, LED_THT:LED_D5.0mm-4_RGB, F.Cu at (153.8, 83.9)
- added U402: SN74LV1T34DBV, Package_TO_SOT_SMD:SOT-23-5, F.Cu at (-18.7, 56.9)
- added U701: AW9523B, Package_DFN_QFN:QFN-24-1EP_4x4mm_P0.5mm_EP2.7x2.7mm, F.Cu at (96.2, 28.6)
- C401: value 100uF 10V -> 100nF; footprint Capacitor_THT:CP_Radial_D6.3mm_P2.50mm -> Capacitor_SMD:C_0603_1608Metric
- R401: value 330K -> 330R; footprint Resistor_SMD:R_1206_3216Metric -> Resistor_SMD:R_0603_1608Metric
- R501, R502, R503, R601, R602, R603: value 4.7K -> 20K
- R701: value 220K -> 4.7K; footprint Resistor_SMD:R_1206_3216Metric -> Resistor_SMD:R_0603_1608Metric
- U101: value ESP32-C3-WROOM-02 -> ESP32-C3-MINI-1; footprint PCM_Espressif:ESP32-C3-WROOM-02 -> PCM_Espressif:ESP32-C3-MINI-1
- U401: value 74HC595 -> CD4504
- U501, U601: value K155ID1 -> HV5222PJ; footprint Package_DIP:DIP-16_W7.62mm -> Package_LCC:PLCC-44_SMD-Socket
- moved C101 131.8 mm to (-23.3, 65.3)
- moved R401 129.9 mm to (-23.3, 60.8)
- moved U401 125.2 mm to (-20.6, 51.2), turned to 0 degrees
- moved R503 117.9 mm to (121.5, 164.3), turned to -90 degrees
- moved R502 111.6 mm to (117.6, 164.3), turned to -90 degrees
- moved R603 107.6 mm to (135.8, 164.3), turned to -90 degrees
- moved R501 106.8 mm to (114.4, 164.3), turned to -90 degrees
- moved R602 102.7 mm to (131.9, 164.3), turned to -90 degrees
- moved R303 100.2 mm to (126.3, 176.4)
- moved R601 100.0 mm to (127.5, 164.3), turned to -90 degrees
- moved R308 98.5 mm to (104.4, 174.9), turned to 90 degrees
- moved R306 98.5 mm to (109.3, 174.9)
- moved R301 98.1 mm to (131.0, 168.6)
- moved C301 98.1 mm to (135.4, 168.6)
- moved C302 98.1 mm to (127.1, 169.0)
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- renumbered C501 to C502, C502 to C503, C503 to C504, C504 to C505, C505 to C506, C506 to C507, C601 to C602, C602 to C603, C603 to C604, C604 to C605, C605 to C606, C606 to C607, J102 to J101, J103 to J102, J101 to J103, TP_107 to TP_101, TP_103 to TP_102, TP_108 to TP_103, TP_109 to TP_104, TP_110 to TP_106, TP_106 to TP_107, TP_104 to TP_108, TP_111 to TP_109
Connections:
- C401 pad 1: GND -> +3V3
- C401 pad 2: +5V -> GND
- C502 pad 1: /Lamps/ThreeDigits1/FIRST_SK6812MINI_VCC -> +5V
- D501 pad 1: /Lamps/ThreeDigits1/FIRST_SK6812MINI_VCC -> +5V
- NX501 pad 0: /Lamps/ThreeDigits1/NX0 -> Net-(U501-HVOUT10)
- NX501 pad 1: /Lamps/ThreeDigits1/NX1 -> Net-(U501-HVOUT1)
- NX501 pad 2: /Lamps/ThreeDigits1/NX2 -> Net-(U501-HVOUT2)
- NX501 pad 3: /Lamps/ThreeDigits1/NX3 -> Net-(U501-HVOUT3)
- NX501 pad 4: /Lamps/ThreeDigits1/NX4 -> Net-(U501-HVOUT4)
- NX501 pad 5: /Lamps/ThreeDigits1/NX5 -> Net-(U501-HVOUT5)
- NX501 pad 6: /Lamps/ThreeDigits1/NX6 -> Net-(U501-HVOUT6)
- NX501 pad 7: /Lamps/ThreeDigits1/NX7 -> Net-(U501-HVOUT7)
- NX501 pad 8: /Lamps/ThreeDigits1/NX8 -> Net-(U501-HVOUT8)
- NX501 pad 9: /Lamps/ThreeDigits1/NX9 -> Net-(U501-HVOUT9)
- NX502 pad 0: /Lamps/ThreeDigits1/NX0 -> Net-(U501-HVOUT20)
- NX502 pad 1: /Lamps/ThreeDigits1/NX1 -> Net-(U501-HVOUT11)
- NX502 pad 2: /Lamps/ThreeDigits1/NX2 -> Net-(U501-HVOUT12)
- NX502 pad 3: /Lamps/ThreeDigits1/NX3 -> Net-(U501-HVOUT13)
- NX502 pad 4: /Lamps/ThreeDigits1/NX4 -> Net-(U501-HVOUT14)
- NX502 pad 5: /Lamps/ThreeDigits1/NX5 -> Net-(U501-HVOUT15)
- NX502 pad 6: /Lamps/ThreeDigits1/NX6 -> Net-(U501-HVOUT16)
- NX502 pad 7: /Lamps/ThreeDigits1/NX7 -> Net-(U501-HVOUT17)
- NX502 pad 8: /Lamps/ThreeDigits1/NX8 -> Net-(U501-HVOUT18)
- NX502 pad 9: /Lamps/ThreeDigits1/NX9 -> Net-(U501-HVOUT19)
- NX503 pad 0: /Lamps/ThreeDigits1/NX0 -> Net-(U501-HVOUT32)
- NX503 pad 1: /Lamps/ThreeDigits1/NX1 -> Net-(U501-HVOUT23)
- NX503 pad 2: /Lamps/ThreeDigits1/NX2 -> Net-(U501-HVOUT24)
- NX503 pad 3: /Lamps/ThreeDigits1/NX3 -> Net-(U501-HVOUT25)
- NX503 pad 4: /Lamps/ThreeDigits1/NX4 -> Net-(U501-HVOUT26)
- NX503 pad 5: /Lamps/ThreeDigits1/NX5 -> Net-(U501-HVOUT27)
- NX503 pad 6: /Lamps/ThreeDigits1/NX6 -> Net-(U501-HVOUT28)
- NX503 pad 7: /Lamps/ThreeDigits1/NX7 -> Net-(U501-HVOUT29)
- NX503 pad 8: /Lamps/ThreeDigits1/NX8 -> Net-(U501-HVOUT30)
- NX503 pad 9: /Lamps/ThreeDigits1/NX9 -> Net-(U501-HVOUT31)
- NX601 pad 0: /Lamps/ThreeDigits2/NX0 -> Net-(U601-HVOUT10)
- NX601 pad 1: /Lamps/ThreeDigits2/NX1 -> Net-(U601-HVOUT1)
- NX601 pad 2: /Lamps/ThreeDigits2/NX2 -> Net-(U601-HVOUT2)
- NX601 pad 3: /Lamps/ThreeDigits2/NX3 -> Net-(U601-HVOUT3)
- NX601 pad 4: /Lamps/ThreeDigits2/NX4 -> Net-(U601-HVOUT4)
- NX601 pad 5: /Lamps/ThreeDigits2/NX5 -> Net-(U601-HVOUT5)
- NX601 pad 6: /Lamps/ThreeDigits2/NX6 -> Net-(U601-HVOUT6)
- NX601 pad 7: /Lamps/ThreeDigits2/NX7 -> Net-(U601-HVOUT7)
- NX601 pad 8: /Lamps/ThreeDigits2/NX8 -> Net-(U601-HVOUT8)
- NX601 pad 9: /Lamps/ThreeDigits2/NX9 -> Net-(U601-HVOUT9)
- NX602 pad 0: /Lamps/ThreeDigits2/NX0 -> Net-(U601-HVOUT20)
- NX602 pad 1: /Lamps/ThreeDigits2/NX1 -> Net-(U601-HVOUT11)
- NX602 pad 2: /Lamps/ThreeDigits2/NX2 -> Net-(U601-HVOUT12)
- NX602 pad 3: /Lamps/ThreeDigits2/NX3 -> Net-(U601-HVOUT13)
- NX602 pad 4: /Lamps/ThreeDigits2/NX4 -> Net-(U601-HVOUT14)
- NX602 pad 5: /Lamps/ThreeDigits2/NX5 -> Net-(U601-HVOUT15)
- NX602 pad 6: /Lamps/ThreeDigits2/NX6 -> Net-(U601-HVOUT16)
- NX602 pad 7: /Lamps/ThreeDigits2/NX7 -> Net-(U601-HVOUT17)
- NX602 pad 8: /Lamps/ThreeDigits2/NX8 -> Net-(U601-HVOUT18)
- NX602 pad 9: /Lamps/ThreeDigits2/NX9 -> Net-(U601-HVOUT19)
- NX603 pad 0: /Lamps/ThreeDigits2/NX0 -> Net-(U601-HVOUT32)
- NX603 pad 1: /Lamps/ThreeDigits2/NX1 -> Net-(U601-HVOUT23)
- NX603 pad 2: /Lamps/ThreeDigits2/NX2 -> Net-(U601-HVOUT24)
- NX603 pad 3: /Lamps/ThreeDigits2/NX3 -> Net-(U601-HVOUT25)
- NX603 pad 4: /Lamps/ThreeDigits2/NX4 -> Net-(U601-HVOUT26)
- NX603 pad 5: /Lamps/ThreeDigits2/NX5 -> Net-(U601-HVOUT27)
- NX603 pad 6: /Lamps/ThreeDigits2/NX6 -> Net-(U601-HVOUT28)
- NX603 pad 7: /Lamps/ThreeDigits2/NX7 -> Net-(U601-HVOUT29)
- NX603 pad 8: /Lamps/ThreeDigits2/NX8 -> Net-(U601-HVOUT30)
- NX603 pad 9: /Lamps/ThreeDigits2/NX9 -> Net-(U601-HVOUT31)
- R401 pad 2: Net-(N401-C) -> /Lamps/ThreeDigits1/SK6812MINI_IN
- R501 pad 2: /Lamps/HighSideSwitch3/VOUT -> +170V
- R502 pad 2: /Lamps/HighSideSwitch2/VOUT -> +170V
- R503 pad 2: /Lamps/HighSideSwitch1/VOUT -> +170V
- R601 pad 2: /Lamps/HighSideSwitch3/VOUT -> +170V
- R602 pad 2: /Lamps/HighSideSwitch2/VOUT -> +170V
- R603 pad 2: /Lamps/HighSideSwitch1/VOUT -> +170V
- R701 pad 1: +170V -> +3V3
- U101 pad 1: +3V3 -> GND
- U101 pad 10: CS -> unconnected-(U101-NC-Pad10)
- U101 pad 11: INPUT -> GND
- U101 pad 12: SK6812MINI_DATA -> unconnected-(U101-GPIO0/ADC1_CH0/XTAL_32K_P-Pad12)
- U101 pad 13: USB_D- -> unconnected-(U101-GPIO1/ADC1_CH1/XTAL_32K_N-Pad13)
- U101 pad 14: USB_D+ -> GND
- U101 pad 15: MUX3 -> unconnected-(U101-NC-Pad15)
- U101 pad 16: DALLAS -> LAMPS_EN
- U101 pad 17: MUX2 -> unconnected-(U101-NC-Pad17)
- U101 pad 18: MUX1 -> unconnected-(U101-GPIO4/ADC1_CH4-Pad18)
- U101 pad 19: GND -> unconnected-(U101-GPIO5/ADC2_CH0-Pad19)
- U101 pad 2: EN -> GND
- U101 pad 3: DBG -> +3V3
- U101 pad 4: COLONS -> unconnected-(U101-NC-Pad4)
- U101 pad 5: SCK -> DALLAS
- U101 pad 6: MOSI -> unconnected-(U101-GPIO3/ADC1_CH3-Pad6)
- U101 pad 7: SDA -> unconnected-(U101-NC-Pad7)
- U101 pad 8: SCL -> EN
- U101 pad 9: GND -> unconnected-(U101-NC-Pad9)
- U401 pad 1: /Lamps/ThreeDigits1/DIGIT_B -> +3V3
- U401 pad 10: +3V3 -> unconnected-(U401-Dout-Pad10)
- U401 pad 11: SCK -> GND
- U401 pad 12: CS -> unconnected-(U401-Eout-Pad12)
- U401 pad 13: GND -> +3V3
- U401 pad 14: MOSI -> GND
- U401 pad 15: /Lamps/ThreeDigits1/DIGIT_A -> unconnected-(U401-Fout-Pad15)
- U401 pad 16: +3V3 -> +12V
- U401 pad 2: /Lamps/ThreeDigits1/DIGIT_C -> /Lamps/ThreeDigits1/CLK
- U401 pad 3: /Lamps/ThreeDigits1/DIGIT_D -> LAMPS_CLK
- U401 pad 4: /Lamps/ThreeDigits2/DIGIT_A -> /Lamps/ThreeDigits1/EN
- U401 pad 5: /Lamps/ThreeDigits2/DIGIT_B -> LAMPS_EN
- U401 pad 6: /Lamps/ThreeDigits2/DIGIT_C -> /Lamps/ThreeDigits1/DATAIN
- U401 pad 7: /Lamps/ThreeDigits2/DIGIT_D -> LAMPS_DATAIN
- U401 pad 9: unconnected-(U401-QH'-Pad9) -> GND
- U501 pad 1: /Lamps/ThreeDigits1/NX8 -> Net-(U501-HVOUT17)
- U501 pad 10: /Lamps/ThreeDigits1/NX7 -> Net-(U501-HVOUT8)
- U501 pad 11: /Lamps/ThreeDigits1/NX6 -> Net-(U501-HVOUT7)
- U501 pad 12: GND -> Net-(U501-HVOUT6)
- U501 pad 13: /Lamps/ThreeDigits1/NX4 -> Net-(U501-HVOUT5)
- U501 pad 14: /Lamps/ThreeDigits1/NX5 -> Net-(U501-HVOUT4)
- U501 pad 15: /Lamps/ThreeDigits1/NX1 -> Net-(U501-HVOUT3)
- U501 pad 16: /Lamps/ThreeDigits1/NX0 -> Net-(U501-HVOUT2)
- U501 pad 2: /Lamps/ThreeDigits1/NX9 -> Net-(U501-HVOUT16)
- U501 pad 3: /Lamps/ThreeDigits1/DIGIT_A -> Net-(U501-HVOUT15)
- U501 pad 4: /Lamps/ThreeDigits1/DIGIT_D -> Net-(U501-HVOUT14)
- U501 pad 5: +5V -> Net-(U501-HVOUT13)
- U501 pad 6: /Lamps/ThreeDigits1/DIGIT_B -> Net-(U501-HVOUT12)
- U501 pad 7: /Lamps/ThreeDigits1/DIGIT_C -> Net-(U501-HVOUT11)
- U501 pad 8: /Lamps/ThreeDigits1/NX2 -> Net-(U501-HVOUT10)
- U501 pad 9: /Lamps/ThreeDigits1/NX3 -> Net-(U501-HVOUT9)
- U601 pad 1: /Lamps/ThreeDigits2/NX8 -> Net-(U601-HVOUT17)
- U601 pad 10: /Lamps/ThreeDigits2/NX7 -> Net-(U601-HVOUT8)
- U601 pad 11: /Lamps/ThreeDigits2/NX6 -> Net-(U601-HVOUT7)
- U601 pad 12: GND -> Net-(U601-HVOUT6)
- U601 pad 13: /Lamps/ThreeDigits2/NX4 -> Net-(U601-HVOUT5)
- U601 pad 14: /Lamps/ThreeDigits2/NX5 -> Net-(U601-HVOUT4)
- U601 pad 15: /Lamps/ThreeDigits2/NX1 -> Net-(U601-HVOUT3)
- U601 pad 16: /Lamps/ThreeDigits2/NX0 -> Net-(U601-HVOUT2)
- U601 pad 2: /Lamps/ThreeDigits2/NX9 -> Net-(U601-HVOUT16)
- U601 pad 3: /Lamps/ThreeDigits2/DIGIT_A -> Net-(U601-HVOUT15)
- U601 pad 4: /Lamps/ThreeDigits2/DIGIT_D -> Net-(U601-HVOUT14)
- U601 pad 5: +5V -> Net-(U601-HVOUT13)
- U601 pad 6: /Lamps/ThreeDigits2/DIGIT_B -> Net-(U601-HVOUT12)
- U601 pad 7: /Lamps/ThreeDigits2/DIGIT_C -> Net-(U601-HVOUT11)
- U601 pad 8: /Lamps/ThreeDigits2/NX2 -> Net-(U601-HVOUT10)
- U601 pad 9: /Lamps/ThreeDigits2/NX3 -> Net-(U601-HVOUT9)
Routing:
- net +5V: track 394.6 -> 0.00 mm, vias 18 -> 0
- net +3V3: track 192.5 -> 0.00 mm, vias 9 -> 0
- net +170V: track 184.6 -> 0.00 mm, vias 8 -> 0
- net MUX1: track 168.9 -> 0.00 mm, vias 2 -> 0
- net GND: track 162.5 -> 0.00 mm, vias 18 -> 0
- net MUX2: track 145.5 -> 0.00 mm, vias 2 -> 0
- net Net-(NX501-PadA): track 114.7 -> 0.00 mm, vias 3 -> 0
- net MUX3: track 112.6 -> 0.00 mm, vias 2 -> 0
- net /Lamps/ThreeDigits2/NX0: track 110.6 -> 0.00 mm, vias 3 -> 0
- net /Lamps/ThreeDigits1/NX2: track 107.4 -> 0.00 mm, vias 1 -> 0
- net /Lamps/ThreeDigits1/NX3: track 104.8 -> 0.00 mm, vias 1 -> 0
- net /Lamps/ThreeDigits2/NX1: track 104.3 -> 0.00 mm, vias 1 -> 0
- net /Lamps/ThreeDigits1/NX1: track 100.7 -> 0.00 mm, vias 1 -> 0
- net /Lamps/ThreeDigits2/NX9: track 100.3 -> 0.00 mm, vias 2 -> 0
- net /Lamps/ThreeDigits2/NX8: track 98.6 -> 0.00 mm, vias 2 -> 0
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Other:
- board size 142 x 61.5 mm -> 146.2 x 64.5 mm

Commit message: almost ready but need to redesign
Parts:
- removed NT302: NetTie_2, NetTie:NetTie-2_SMD_Pad0.5mm
- removed R106: 4.7K, Resistor_SMD:R_0603_1608Metric
- removed U102: DS18B20, Package_TO_SOT_THT:TO-92_Inline
- added NT106: NetTie_2, NetTie:NetTie-2_SMD_Pad0.5mm, F.Cu at (114.9, 116.0)
- BT101, J102, J103, J104: moved to B.Cu
- D701, D702, D703, D704: footprint LED_THT:LED_D5.0mm-4_RGB -> LED_THT:LED_D5.0mm-4_RGB_Wide_Pins
- TP_105: value SDA -> SDA/BOOT
- moved C601 180.0 mm to (150.7, 116.0), turned to 180 degrees
- moved C501 142.4 mm to (113.1, 115.5), turned to 90 degrees
- moved U103 121.5 mm to (81.9, 64.7), turned to 180 degrees
- moved C101 120.3 mm to (84.9, 118.0), turned to -90 degrees
- moved J102 116.8 mm to (97.0, 63.6)
- moved C402 116.1 mm to (84.5, 101.4)
- moved C401 115.7 mm to (84.3, 98.2)
- moved C103 114.0 mm to (88.0, 63.4), turned to 90 degrees
- moved U401 110.0 mm to (78.6, 98.9)
- moved TP_105 103.8 mm to (186.0, 62.0)
- moved R401 99.8 mm to (76.5, 63.4), turned to 90 degrees
- moved TP_107 97.8 mm to (186.0, 64.5)
- moved NT301 97.0 mm to (148.7, 95.6), turned to 90 degrees
- moved BT101 95.6 mm to (99.0, 99.9), turned to -90 degrees
- moved U402 91.0 mm to (72.0, 63.8)
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Connections:
- net Net-(R306-Pad2) renamed /UC3843/PWR_R
- net Net-(U501-HVOUT1) renamed /Lamps/ThreeDigits1/LAMP_C1.1
- net Net-(U501-HVOUT10) renamed /Lamps/ThreeDigits1/LAMP_C1.0
- net Net-(U501-HVOUT11) renamed /Lamps/ThreeDigits1/LAMP_C2.1
- net Net-(U501-HVOUT12) renamed /Lamps/ThreeDigits1/LAMP_C2.2
- net Net-(U501-HVOUT13) renamed /Lamps/ThreeDigits1/LAMP_C2.3
- net Net-(U501-HVOUT14) renamed /Lamps/ThreeDigits1/LAMP_C2.4
- net Net-(U501-HVOUT15) renamed /Lamps/ThreeDigits1/LAMP_C2.5
- net Net-(U501-HVOUT16) renamed /Lamps/ThreeDigits1/LAMP_C2.6
- net Net-(U501-HVOUT17) renamed /Lamps/ThreeDigits1/LAMP_C2.7
- net Net-(U501-HVOUT18) renamed /Lamps/ThreeDigits1/LAMP_C2.8
- net Net-(U501-HVOUT19) renamed /Lamps/ThreeDigits1/LAMP_C2.9
- net Net-(U501-HVOUT2) renamed /Lamps/ThreeDigits1/LAMP_C1.2
- net Net-(U501-HVOUT20) renamed /Lamps/ThreeDigits1/LAMP_C2.0
- net Net-(U501-HVOUT23) renamed /Lamps/ThreeDigits1/LAMP_C3.1
- net Net-(U501-HVOUT24) renamed /Lamps/ThreeDigits1/LAMP_C3.2
- net Net-(U501-HVOUT25) renamed /Lamps/ThreeDigits1/LAMP_C3.3
- net Net-(U501-HVOUT26) renamed /Lamps/ThreeDigits1/LAMP_C3.4
- net Net-(U501-HVOUT27) renamed /Lamps/ThreeDigits1/LAMP_C3.5
- net Net-(U501-HVOUT28) renamed /Lamps/ThreeDigits1/LAMP_C3.6
- net Net-(U501-HVOUT29) renamed /Lamps/ThreeDigits1/LAMP_C3.7
- net Net-(U501-HVOUT3) renamed /Lamps/ThreeDigits1/LAMP_C1.3
- net Net-(U501-HVOUT30) renamed /Lamps/ThreeDigits1/LAMP_C3.8
- net Net-(U501-HVOUT31) renamed /Lamps/ThreeDigits1/LAMP_C3.9
- net Net-(U501-HVOUT32) renamed /Lamps/ThreeDigits1/LAMP_C3.0
- net Net-(U501-HVOUT4) renamed /Lamps/ThreeDigits1/LAMP_C1.4
- net Net-(U501-HVOUT5) renamed /Lamps/ThreeDigits1/LAMP_C1.5
- net Net-(U501-HVOUT6) renamed /Lamps/ThreeDigits1/LAMP_C1.6
- net Net-(U501-HVOUT7) renamed /Lamps/ThreeDigits1/LAMP_C1.7
- net Net-(U501-HVOUT8) renamed /Lamps/ThreeDigits1/LAMP_C1.8
- net Net-(U501-HVOUT9) renamed /Lamps/ThreeDigits1/LAMP_C1.9
- net Net-(U601-HVOUT1) renamed /Lamps/ThreeDigits2/LAMP_C1.1
- net Net-(U601-HVOUT10) renamed /Lamps/ThreeDigits2/LAMP_C1.0
- net Net-(U601-HVOUT11) renamed /Lamps/ThreeDigits2/LAMP_C2.1
- net Net-(U601-HVOUT12) renamed /Lamps/ThreeDigits2/LAMP_C2.2
- net Net-(U601-HVOUT13) renamed /Lamps/ThreeDigits2/LAMP_C2.3
- net Net-(U601-HVOUT14) renamed /Lamps/ThreeDigits2/LAMP_C2.4
- net Net-(U601-HVOUT15) renamed /Lamps/ThreeDigits2/LAMP_C2.5
- net Net-(U601-HVOUT16) renamed /Lamps/ThreeDigits2/LAMP_C2.6
- net Net-(U601-HVOUT17) renamed /Lamps/ThreeDigits2/LAMP_C2.7
- net Net-(U601-HVOUT18) renamed /Lamps/ThreeDigits2/LAMP_C2.8
- net Net-(U601-HVOUT19) renamed /Lamps/ThreeDigits2/LAMP_C2.9
- net Net-(U601-HVOUT2) renamed /Lamps/ThreeDigits2/LAMP_C1.2
- net Net-(U601-HVOUT20) renamed /Lamps/ThreeDigits2/LAMP_C2.0
- net Net-(U601-HVOUT23) renamed /Lamps/ThreeDigits2/LAMP_C3.1
- net Net-(U601-HVOUT24) renamed /Lamps/ThreeDigits2/LAMP_C3.2
- net Net-(U601-HVOUT25) renamed /Lamps/ThreeDigits2/LAMP_C3.3
- net Net-(U601-HVOUT26) renamed /Lamps/ThreeDigits2/LAMP_C3.4
- net Net-(U601-HVOUT27) renamed /Lamps/ThreeDigits2/LAMP_C3.5
- net Net-(U601-HVOUT28) renamed /Lamps/ThreeDigits2/LAMP_C3.6
- net Net-(U601-HVOUT29) renamed /Lamps/ThreeDigits2/LAMP_C3.7
- net Net-(U601-HVOUT3) renamed /Lamps/ThreeDigits2/LAMP_C1.3
- net Net-(U601-HVOUT30) renamed /Lamps/ThreeDigits2/LAMP_C3.8
- net Net-(U601-HVOUT31) renamed /Lamps/ThreeDigits2/LAMP_C3.9
- net Net-(U601-HVOUT32) renamed /Lamps/ThreeDigits2/LAMP_C3.0
- net Net-(U601-HVOUT4) renamed /Lamps/ThreeDigits2/LAMP_C1.4
- net Net-(U601-HVOUT5) renamed /Lamps/ThreeDigits2/LAMP_C1.5
- net Net-(U601-HVOUT6) renamed /Lamps/ThreeDigits2/LAMP_C1.6
- net Net-(U601-HVOUT7) renamed /Lamps/ThreeDigits2/LAMP_C1.7
- net Net-(U601-HVOUT8) renamed /Lamps/ThreeDigits2/LAMP_C1.8
- net Net-(U601-HVOUT9) renamed /Lamps/ThreeDigits2/LAMP_C1.9
- C205 pad 1: +12V -> /MP2307/+12V
- C206 pad 1: +12V -> /MP2307/+12V
- C304 pad 1: +12V -> /MP2307/+12V
- J104 pad 2: +12V -> /MP2307/+12V
- L301 pad 1: +12V -> /MP2307/+12V
- NT201 pad 1: +12V -> /MP2307/+12V
- NT301 pad 2: +12V -> /MP2307/+12V
- R303 pad 1: Net-(NT302-Pad2) -> +170V
- U101 pad 5: DALLAS -> unconnected-(U101-GPIO2/ADC1_CH2-Pad5)
- U202 pad 2: +12V -> /MP2307/+12V
- U701 pad 1: Net-(D703-RK) -> Net-(D703-GK)
- U701 pad 10: Net-(D702-GK) -> Net-(D701-BK)
- U701 pad 11: Net-(D702-BK) -> Net-(D702-RK)
- U701 pad 12: unconnected-(U701-P0_6-Pad12) -> Net-(D702-GK)
- U701 pad 13: unconnected-(U701-P0_7-Pad13) -> Net-(D702-BK)
- U701 pad 14: Net-(D704-GK) -> Net-(D703-RK)
- U701 pad 15: Net-(D704-BK) -> Net-(D704-RK)
- U701 pad 16: unconnected-(U701-P1_6-Pad16) -> Net-(D704-GK)
- U701 pad 17: unconnected-(U701-P1_7-Pad17) -> Net-(D704-BK)
- U701 pad 2: Net-(D703-GK) -> Net-(D703-BK)
- U701 pad 3: Net-(D703-BK) -> unconnected-(U701-P1_2-Pad3)
- U701 pad 4: Net-(D704-RK) -> unconnected-(U701-P1_3-Pad4)
- U701 pad 5: Net-(D701-RK) -> unconnected-(U701-P0_0-Pad5)
- U701 pad 6: Net-(D701-GK) -> unconnected-(U701-P0_1-Pad6)
- U701 pad 7: Net-(D701-BK) -> Net-(D701-RK)
- U701 pad 8: Net-(D702-RK) -> Net-(D701-GK)
Routing:
- net +5V: track 0.00 -> 419.4 mm, vias 0 -> 4
- net SCL: track 0.00 -> 194.7 mm, vias 0 -> 6
- net SDA: track 0.00 -> 187.8 mm, vias 0 -> 2
- net /MP2307/+12V: track 0.00 -> 160.3 mm, vias 0 -> 1
- net +12V: track 0.00 -> 142.2 mm, vias 0 -> 5
- net /Lamps/ThreeDigits1/CLK: track 0.00 -> 110.2 mm, vias 0 -> 3
- net /Lamps/ThreeDigits1/EN: track 0.00 -> 106.5 mm, vias 0 -> 3
- net /UC3843/PWR_GND: track 0.00 -> 87.9 mm, vias 0 -> 2
- net /Lamps/ThreeDigits1/DATAOUT: track 0.00 -> 82.7 mm, vias 0 -> 2
- net INPUT: track 0.00 -> 77.9 mm, vias 0 -> 1
- net Net-(D702-RK): track 0.00 -> 68.1 mm, vias 0 -> 1
- net +3V3: track 0.00 -> 65.0 mm
- net Net-(D702-GK): track 0.00 -> 59.8 mm, vias 0 -> 1
- net Net-(D702-BK): track 0.00 -> 58.8 mm, vias 0 -> 1
- net Net-(D701-RK): track 0.00 -> 58.0 mm, vias 0 -> 1
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Other:
- board size 146.2 x 64.5 mm -> 144 x 60 mm
- board text added: "12VIN"
- board text added: "v2.0"
- board text removed: "IN12V"
- board text removed: "v1.0"

Commit message: connect all
Parts:
- removed NT102, NT103: NetTie_2, NetTie:NetTie-2_SMD_Pad0.5mm
- added TP_110: GND, NosLib:TestPoint_Pad_1.0x1.0mm, F.Cu at (191.8, 64.3)
- moved NT203 4.42 mm to (197.6, 112.1)
- moved NT301 1.54 mm to (150.3, 95.7)
- moved C501 1.39 mm to (113.1, 114.1)
- moved NT101 0.74 mm to (65.0, 98.0), turned to 180 degrees
- moved C603 0.20 mm to (145.8, 82.6)
- moved C607 0.19 mm to (195.7, 82.6)
- moved C605 0.17 mm to (175.6, 82.5)
- moved C507 0.14 mm to (125.6, 82.5)
- moved C505 0.13 mm to (95.8, 82.5)
- moved U101 0.13 mm to (76.5, 110.9)
- turned C301 to 180 degrees
- turned C502 to 90 degrees
- turned C504 to 90 degrees
- turned C506 to 90 degrees
- turned C602 to 90 degrees
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Connections:
- C202 pad 1: /MP2307/+5V -> +5V
- C203 pad 1: /MP2307/+3V3 -> +3V3
- C204 pad 1: /MP2307/+3V3 -> +3V3
- C207 pad 1: /MP2307/+5V -> +5V
- C208 pad 1: /MP2307/+5V -> +5V
- L201 pad 2: /MP2307/+5V -> +5V
- NT202 pad 2: /MP2307/+5V -> +5V
- U201 pad 2: /MP2307/+3V3 -> +3V3
- U201 pad 3: /MP2307/+5V -> +5V
Routing:
- net +3V3: track 65.0 -> 350.9 mm, vias 0 -> 10
- net GND: track 11.3 -> 169.1 mm, vias 0 -> 21
- net Net-(NX603-PadA): track 0.00 -> 66.5 mm
- net Net-(NX602-PadA): track 0.00 -> 50.2 mm
- net Net-(NX501-PadA): track 0.00 -> 40.9 mm
- net +170V: track 17.2 -> 50.2 mm
- net /MP2307/+5V: track 30.0 -> 0.00 mm
- net Net-(NX502-PadA): track 0.00 -> 24.6 mm
- net Net-(NX601-PadA): track 0.00 -> 24.2 mm
- net +5V: track 419.4 -> 403.1 mm, vias 4 -> 6
- net /MP2307/+3V3: track 13.7 -> 0.00 mm
- net SDA: track 187.8 -> 200.3 mm, vias 2 -> 4
- net EN: track 0.00 -> 11.0 mm
- net Net-(Q301-G): track 0.00 -> 10.5 mm, vias 0 -> 2
- net Net-(NX503-PadA): track 0.00 -> 9.76 mm
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