File: hardware/ThreeDigits.kicad_sch (KiCad schematic)
At the start: 19 parts, among them U501 K155ID1

Commit message: Finalize schematics
Parts:
- NX501, NX502, NX503: footprint nixies-us:nixies-us-IN-12 -> NosLib:nixies-us-IN-12
- R501, R502, R503: value 22K -> 4.7K; footprint Resistor_SMD:R_2512_6332Metric -> Resistor_SMD:R_1206_3216Metric
Changed lines of the file:
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@@
 			)
 		)
-		(property "Value" "22K"
+		(property "Value" "4.7K"
 			(at 121.92 125.73 90)
 			(effects
@@
 			)
 		)
-		(property "Footprint" "Resistor_SMD:R_2512_6332Metric"
+		(property "Footprint" "Resistor_SMD:R_1206_3216Metric"
 			(at 121.92 131.318 90)
 			(effects
@@
 			)
 		)
-		(property "Footprint" "nixies-us:nixies-us-IN-12"
+		(property "Footprint" "NosLib:nixies-us-IN-12"
 			(at 107.95 88.9 0)
 			(effects
@@
 			)
 		)
-		(property "Footprint" "nixies-us:nixies-us-IN-12"
+		(property "Footprint" "NosLib:nixies-us-IN-12"
 			(at 106.68 48.26 0)
 			(effects
@@
 			)
 		)
-		(property "Value" "22K"
+		(property "Value" "4.7K"
 			(at 120.65 44.45 90)
 			(effects
@@
 			)
 		)
-		(property "Footprint" "Resistor_SMD:R_2512_6332Metric"
+		(property "Footprint" "Resistor_SMD:R_1206_3216Metric"
 			(at 120.65 50.038 90)
 			(effects
@@
 			)
 		)
-		(property "Value" "22K"
+		(property "Value" "4.7K"
 			(at 121.92 85.09 90)
 			(effects
@@
 			)
 		)
-		(property "Footprint" "Resistor_SMD:R_2512_6332Metric"
+		(property "Footprint" "Resistor_SMD:R_1206_3216Metric"
 			(at 121.92 90.678 90)
 			(effects
@@
 			)
 		)
-		(property "Footprint" "nixies-us:nixies-us-IN-12"
+		(property "Footprint" "NosLib:nixies-us-IN-12"
 			(at 107.95 129.54 0)
 			(effects

Commit message: Fixes
Parts:
- NX501, NX502, NX503: footprint NosLib:nixies-us-IN-12 -> nixies-us:IN-12
Changed lines of the file:
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@@
 			)
 		)
-		(property "Footprint" "NosLib:nixies-us-IN-12"
+		(property "Footprint" "nixies-us:IN-12"
 			(at 107.95 88.9 0)
 			(effects
@@
 			)
 		)
-		(property "Footprint" "NosLib:nixies-us-IN-12"
+		(property "Footprint" "nixies-us:IN-12"
 			(at 106.68 48.26 0)
 			(effects
@@
 			)
 		)
-		(property "Footprint" "NosLib:nixies-us-IN-12"
+		(property "Footprint" "nixies-us:IN-12"
 			(at 107.95 129.54 0)
 			(effects
