File: hardware/ThreeDigits.kicad_sch (KiCad schematic)
At the start: 20 parts, among them U501 HV5222PJ

Commit message: almost ready but need to redesign
Connections:
- net LAMP_C2.0: now reaches NX502.0, U501.42 (HVOUT20)
- net LAMP_C2.1: now reaches NX502.1, U501.7 (HVOUT11)
- net LAMP_C2.2: now reaches NX502.2, U501.6 (HVOUT12)
- net LAMP_C2.3: now reaches NX502.3, U501.5 (HVOUT13)
- net LAMP_C2.4: now reaches NX502.4, U501.4 (HVOUT14)
- net LAMP_C2.5: now reaches NX502.5, U501.3 (HVOUT15)
- net LAMP_C2.6: now reaches NX502.6, U501.2 (HVOUT16)
- net LAMP_C2.7: now reaches NX502.7, U501.1 (HVOUT17)
- net LAMP_C2.8: now reaches NX502.8, U501.44 (HVOUT18)
- net LAMP_C2.9: now reaches NX502.9, U501.43 (HVOUT19)
- net LAMP_C1.0: now reaches NX501.0, U501.8 (HVOUT10)
- net LAMP_C1.1: now reaches NX501.1, U501.17 (HVOUT1)
- net LAMP_C1.2: now reaches NX501.2, U501.16 (HVOUT2)
- net LAMP_C1.3: now reaches NX501.3, U501.15 (HVOUT3)
- net LAMP_C1.4: now reaches NX501.4, U501.14 (HVOUT4)
- net LAMP_C1.5: now reaches NX501.5, U501.13 (HVOUT5)
- net LAMP_C1.6: now reaches NX501.6, U501.12 (HVOUT6)
- net LAMP_C1.7: now reaches NX501.7, U501.11 (HVOUT7)
- net LAMP_C1.8: now reaches NX501.8, U501.10 (HVOUT8)
- net LAMP_C1.9: now reaches NX501.9, U501.9 (HVOUT9)
- net LAMP_C3.0: now reaches NX503.0, U501.30 (HVOUT32)
- net LAMP_C3.9: now reaches NX503.9, U501.31 (HVOUT31)
- net LAMP_C3.8: now reaches NX503.8, U501.32 (HVOUT30)
- net LAMP_C3.7: now reaches NX503.7, U501.33 (HVOUT29)
- net LAMP_C3.6: now reaches NX503.6, U501.34 (HVOUT28)
- net LAMP_C3.5: now reaches NX503.5, U501.35 (HVOUT27)
- net LAMP_C3.4: now reaches NX503.4, U501.36 (HVOUT26)
- net LAMP_C3.3: now reaches NX503.3, U501.37 (HVOUT25)
- net LAMP_C3.2: now reaches NX503.2, U501.38 (HVOUT24)
- net LAMP_C3.1: now reaches NX503.1, U501.39 (HVOUT23)
