File: hardware/Colons.kicad_sch (KiCad schematic)
At the start: 8 parts, among them U701 AW9523B

Commit message: almost ready but need to redesign
Parts:
- D701, D702, D703, D704: footprint LED_THT:LED_D5.0mm-4_RGB -> LED_THT:LED_D5.0mm-4_RGB_Wide_Pins
Connections:
- net at D703.1 (RK): now also U701.14 (P1_4); no longer U701.1 (P1_0)
- net at D703.3 (GK): now also U701.1 (P1_0); no longer U701.2 (P1_1)
- net at D703.4 (BK): now also U701.2 (P1_1); no longer U701.3 (P1_2)
- net at U701.10 (P0_4): now also D701.4 (BK); no longer D702.3 (GK)
- net at U701.11 (P0_5): now also D702.1 (RK); no longer D702.4 (BK)
- net at U701.12 (P0_6): now also D702.3 (GK)
- net at U701.13 (P0_7): now also D702.4 (BK)
- net at D704.3 (GK): now also U701.16 (P1_6); no longer U701.14 (P1_4)
- net at U701.15 (P1_5): now also D704.1 (RK); no longer D704.4 (BK)
- net at U701.17 (P1_7): now also D704.4 (BK)
- net at U701.4 (P1_3): no longer D704.1 (RK)
- net at U701.5 (P0_0): no longer D701.1 (RK)
- net at U701.6 (P0_1): no longer D701.3 (GK)
- net at U701.7 (P0_2): now also D701.1 (RK); no longer D701.4 (BK)
- net at U701.8 (P0_3): now also D701.3 (GK); no longer D702.1 (RK)
