File: hardware/MP2307.kicad_sch (KiCad schematic)
At the start: 17 parts, among them U201 MP2307DN-LF-Z

Commit message: Static version (incomplete)
Parts:
- C204: footprint Capacitor_SMD:C_0805_2012Metric -> Capacitor_SMD:C_0603_1608Metric
- renumbered C207 to C209, R202 to R204, R203 to R205, R204 to R206, U201 to U203
Other:
- moved on the sheet: C201, C209

Commit message: 2/static version
Parts:
- added C202, C203: 100nF, Capacitor_SMD:C_0603_1608Metric, symbol Device:C
- added C204: 10uF, Capacitor_SMD:C_0805_2012Metric, symbol Device:C
- added U201: AP7361-33ER-13, Package_TO_SOT_SMD:SOT-223-3_TabPin2, symbol Regulator_Linear:AMS1117-3.3
- renumbered C205 to C201, C201 to C205, C202 to C206, C206 to C207, C209 to C208, C203 to C209, C204 to C210, NT203 to NT202, NT204 to NT203, NT202 to NT204, R206 to R202, R205 to R203, U203 to U202
Connections:
- net +5V: now also C202.1, U201.3 (VI)
- net GND: now also C202.2, C203.2, C204.2, U201.1 (GND); no longer U202.4 (GND)
- net PWR_GND: now also U202.4 (GND)
- new net +3V3: C203.1, C204.1, U201.2 (VO)
Other:
- moved on the sheet: C201, C205, C206, C207, C208, C209, C210, L201, NT201, NT202, NT203, NT204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

Commit message: Finalize schematics
Parts:
- removed NT202: NetTie_SW_BS, NetTie:NetTie-2_SMD_Pad0.5mm, symbol Device:NetTie_2
- renumbered NT203 to NT202, NT204 to NT203
Connections:
- net SW: now also C201.2
Other:
- note added: "Vout = 0.925 * (1 + Rtop / Rbottom) = 0.925 * (1 + 30K / 6,8K) = 5.005V"
- note removed: "Vout = 0.925 * (1 + R204 / R203) = 0.925 * (1 + 30K / 6,8K) = 5.005V"
- moved on the sheet: C202, C203, C204, U201
